File: schematics/kicad/pico-glitcher.kicad_pcb (KiCad board)
At the start: 2 copper layers, 89.8 x 58.4 mm, 72 parts, among them Q1 IRLML2502, Q2 IRF7807PBF, Q3 TPS 79318, Q4 TPS2041, U1 NH245, U2 NH245, X1 BU-SMA-V, X2 BU-SMA, X3 M08X2

Commit message: replaced LEDs symbol and footprint with kicad library's ones
Parts:
- D1, D2, D3, D4, D5: footprint pico-glitcher:LED-0603 -> LED_SMD:LED_0603_1608Metric
- moved D2 1.01 mm to (188.9, 124.1), turned to 180 degrees
- moved D3 1.01 mm to (189.0, 126.6), turned to 180 degrees
- moved D4 1.01 mm to (188.9, 121.5), turned to 180 degrees
- moved D1 1.01 mm to (188.9, 131.7), turned to 180 degrees
- moved D5 1.01 mm to (188.9, 129.1), turned to 180 degrees
- moved R6 0.17 mm to (185.0, 124.1)
- moved R8 0.17 mm to (185.0, 126.6)
- moved R9 0.17 mm to (185.0, 121.5)
- moved R10 0.17 mm to (185.0, 129.1)
- moved R7 0.17 mm to (185.0, 131.7)
Connections:
- C1 pad 1: (no net) -> Net-(Q3-NC/FB)
- C2 pad 1: (no net) -> /+1V8
- C7 pad 1: (no net) -> /VTARGET
- JMP_VCC_INTERN0 pad 2: (no net) -> /JVCC
- PICO0 pad 3V3_EN: (no net) -> unconnected-(PICO0-Pad3V3_EN)
- PICO0 pad GP0: (no net) -> /GP0
- PICO0 pad GP1: (no net) -> /GP1
- PICO0 pad GP10: (no net) -> /GP10
- PICO0 pad GP11: (no net) -> /GP11
- PICO0 pad GP12: (no net) -> /GP12
- PICO0 pad GP13: (no net) -> /GP13
- PICO0 pad GP14: (no net) -> /GP14
- PICO0 pad GP15: (no net) -> /GP15
- PICO0 pad GP16: (no net) -> /HPGLITCH2
- PICO0 pad GP17: (no net) -> /LPGLITCH2
- PICO0 pad GP18: (no net) -> Net-(PICO0-PadGP18)
- PICO0 pad GP19: (no net) -> Net-(PICO0-PadGP19)
- PICO0 pad GP2: (no net) -> /GP2
- PICO0 pad GP20: (no net) -> /VTARGET_EN
- PICO0 pad GP21: (no net) -> /VTARGET_OC
- PICO0 pad GP22: (no net) -> unconnected-(PICO0-PadGP22)
- PICO0 pad GP26_A0: (no net) -> /ANALOG
- PICO0 pad GP27_A1: (no net) -> unconnected-(PICO0-PadGP27_A1)
- PICO0 pad GP28_A2: (no net) -> unconnected-(PICO0-PadGP28_A2)
- PICO0 pad GP3: (no net) -> /GP3
- PICO0 pad GP4: (no net) -> /GP4
- PICO0 pad GP5: (no net) -> /GP5
- PICO0 pad GP6: (no net) -> /GP6
- PICO0 pad GP7: (no net) -> /GP7
- PICO0 pad GP8: (no net) -> /GP8
- PICO0 pad GP9: (no net) -> /GP9
- PICO0 pad RUN: (no net) -> Net-(S_RST0-1)
- PICO0 pad SWCLK: (no net) -> unconnected-(PICO0-PadSWCLK)
- PICO0 pad SWDIO: (no net) -> unconnected-(PICO0-PadSWDIO)
- PICO0 pad VSYS: (no net) -> unconnected-(PICO0-PadVSYS)
- Q1 pad 1: (no net) -> Net-(Q1-G)
- Q1 pad 3: (no net) -> Net-(Q1-D)
- Q2 pad 4: (no net) -> Net-(Q2-G)
- R1 pad 1: (no net) -> Net-(U2-DIR)
- R10 pad 1: Net-(D5-PadA) -> Net-(D5-A)
- R12 pad 1: (no net) -> Net-(U1-B1)
- R12 pad 2: (no net) -> Net-(U1-B2)
- R12 pad 3: (no net) -> Net-(U1-B3)
- R12 pad 4: (no net) -> Net-(U1-B4)
- R13 pad 1: (no net) -> Net-(U1-B5)
- R13 pad 2: (no net) -> Net-(U1-B6)
- R13 pad 3: (no net) -> Net-(U1-B7)
- R13 pad 4: (no net) -> Net-(U1-B8)
- R16 pad 5: (no net) -> Net-(U1-A4)
- R16 pad 6: (no net) -> Net-(U1-A3)
- R16 pad 7: (no net) -> Net-(U1-A2)
- R16 pad 8: (no net) -> Net-(U1-A1)
- R17 pad 5: (no net) -> Net-(U1-A8)
- R17 pad 6: (no net) -> Net-(U1-A7)
- R17 pad 7: (no net) -> Net-(U1-A6)
- R17 pad 8: (no net) -> Net-(U1-A5)
- R18 pad 1: (no net) -> Net-(U2-B1)
- R18 pad 2: (no net) -> Net-(U2-B2)
- R18 pad 3: (no net) -> Net-(U2-B3)
- R18 pad 4: (no net) -> Net-(U2-B4)
- R18 pad 5: (no net) -> Net-(R18-Pad5)
- R18 pad 6: (no net) -> Net-(R18-Pad6)
- R18 pad 7: (no net) -> Net-(R18-Pad7)
- R18 pad 8: (no net) -> Net-(R18-Pad8)
- R19 pad 1: (no net) -> Net-(U2-B5)
- R19 pad 2: (no net) -> Net-(U2-B6)
- R19 pad 3: (no net) -> Net-(U2-B7)
- R19 pad 4: (no net) -> Net-(U2-B8)
- R19 pad 5: (no net) -> Net-(R19-Pad5)
- R19 pad 6: (no net) -> Net-(R19-Pad6)
- R19 pad 7: (no net) -> Net-(R19-Pad7)
- R19 pad 8: (no net) -> Net-(R19-Pad8)
- R6 pad 1: Net-(D2-PadA) -> Net-(D2-A)
- R7 pad 1: Net-(D1-PadA) -> Net-(D1-A)
- R8 pad 1: Net-(D3-PadA) -> Net-(D3-A)
- R9 pad 1: Net-(D4-PadA) -> Net-(D4-A)
Routing:
- net Net-(D3-PadA): track 3.51 -> 0.00 mm
- net Net-(D4-PadA): track 3.50 -> 0.00 mm
- net Net-(D1-PadA): track 3.50 -> 0.00 mm
- net Net-(D5-PadA): track 3.35 -> 0.00 mm
- net Net-(D2-PadA): track 3.35 -> 0.00 mm
- net GND: track 67.3 -> 64.8 mm
- net Net-(D3-A): track 0.00 -> 2.29 mm
- net Net-(D5-A): track 0.00 -> 2.27 mm
- net Net-(D4-A): track 0.00 -> 2.27 mm
- net Net-(D2-A): track 0.00 -> 2.27 mm
- net Net-(D1-A): track 0.00 -> 2.27 mm
- net /LPGLITCH2: track 108.6 -> 110.0 mm
Other:
- outline, holes or cut-outs redrawn

Commit message: replaced 0603 resistor's symbol and footprint with kicad library's ones
Parts:
- R1, R10, R11, R2, R3, R4, R5, R6, R7, R8, R9: footprint pico-glitcher:0603-RES -> Resistor_SMD:R_0603_1608Metric
Connections:
- R10 pad 1: Net-(D5-A) -> /HPGLITCH2
- R10 pad 2: /HPGLITCH2 -> Net-(D5-A)
- R2 pad 1: GND -> Net-(Q1-G)
- R2 pad 2: Net-(Q1-G) -> GND
- R4 pad 1: Net-(Q2-G) -> unconnected-(R4-Pad1)
- R4 pad 2: /HPGLITCH2 -> Net-(Q2-G)
- R6 pad 1: Net-(D2-A) -> /GP1
- R6 pad 2: /GP1 -> Net-(D2-A)
- R7 pad 1: Net-(D1-A) -> /LPGLITCH2
- R7 pad 2: /LPGLITCH2 -> Net-(D1-A)
- R8 pad 1: Net-(D3-A) -> /GP15
- R8 pad 2: /GP15 -> Net-(D3-A)
- R9 pad 1: Net-(D4-A) -> /VTARGET
- R9 pad 2: /VTARGET -> Net-(D4-A)

Commit message: replaced 0603 capacitor's symbol and footprint with kicad library's ones
  also: simplified some tracks.
Parts:
- C1, C10, C3, C4, C5, C6, C7, C9: footprint pico-glitcher:0603 -> Capacitor_SMD:C_0603_1608Metric
- moved C4 1.51 mm to (127.1, 113.4), turned to -90 degrees
- moved C5 1.51 mm to (143.6, 113.4), turned to -90 degrees
- moved C6 0.39 mm to (143.6, 110.1)
- moved C3 0.25 mm to (127.1, 109.8)
- turned R6 to 0 degrees
- turned R7 to 0 degrees
- turned R8 to 0 degrees
- turned R9 to 0 degrees
Routing:
- net /GP0: track 44.7 -> 19.7 mm, vias 2 -> 0
- net GND: track 64.8 -> 73.9 mm, vias 8 -> 14
- net /VTARGET: track 83.4 -> 74.8 mm
- net Net-(U1-B8): track 50.0 -> 44.5 mm
- net Net-(R19-Pad5): track 123.7 -> 121.3 mm
- net VCC: track 150.4 -> 148.6 mm
- net Net-(R19-Pad6): track 109.0 -> 107.6 mm
- net /GP4: track 14.1 -> 12.9 mm, vias 2 -> 1
- net /GP1: track 115.4 -> 116.5 mm
- net +3V3: track 150.3 -> 151.1 mm
- net /GP5: track 12.8 -> 12.2 mm

Commit message: replaced 1x03 pinheader's symbol and footprint with kicad library's ones
Parts:
- X_1V8, X_3V3, X_5V0, X_GLITCH_EN0, X_GND0, X_RESET0, X_TRIGGER2, X_VTARGET0: footprint pico-glitcher:1X03 -> Connector_PinHeader_2.54mm:PinHeader_1x03_P2.54mm_Vertical
- turned X_1V8 to 90 degrees
- turned X_3V3 to 90 degrees
- turned X_5V0 to 90 degrees
- turned X_GLITCH_EN0 to 90 degrees
- turned X_GND0 to 90 degrees
- turned X_RESET0 to 90 degrees
- turned X_TRIGGER2 to 90 degrees
- turned X_VTARGET0 to 90 degrees
Connections:
- X_VTARGET0 pad 1: /VTARGET -> unconnected-(X_VTARGET0-Pin_1-Pad1)
- X_VTARGET0 pad 2: /VTARGET -> unconnected-(X_VTARGET0-Pin_2-Pad2)
- X_VTARGET0 pad 3: /VTARGET -> unconnected-(X_VTARGET0-Pin_3-Pad3)
Routing:
- net /VTARGET: track 74.8 -> 72.3 mm
- net +3V3: track 151.1 -> 148.7 mm

Commit message: improved placement and connection of C9
Parts:
- moved C9 0.77 mm to (165.7, 102.2)
Routing:
- net VCC: track 148.6 -> 145.7 mm
- net GND: track 73.9 -> 71.3 mm, vias 14 -> 16
Changed lines of the file:
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@@
 	(footprint "Capacitor_SMD:C_0603_1608Metric"
 		(layer "F.Cu")
-		(at 164.9611 102.1686)
+		(at 165.7351 102.1686)
 		(descr "Capacitor SMD 0603 (1608 Metric), square (rectangular) end terminal, IPC_7351 nominal, (Body size source: IPC-SM-782 page 76, https://www.pcb-3d.com/wordpress/wp-content/uploads/ipc-sm-782a_amendment_1_and_2.pdf), generated with kicad-footprint-generator")
 		(tags "capacitor")
 		(property "Reference" "C9"
-			(at 0 -1.43 0)
+			(at 0 1.56 0)
 			(layer "F.SilkS")
 			(effects
@@
 	)
 	(segment
-		(start 163.2711 101.3286)
-		(end 164.1111 102.1686)
-		(width 0.4064)
-		(layer "F.Cu")
-		(net 3)
-	)
-	(segment
 		(start 140.1461 114.7156)
 		(end 141.0971 115.6666)
@@
 	)
 	(segment
-		(start 163.2711 101.1886)
-		(end 163.2711 101.3286)
-		(width 0.4064)
-		(layer "F.Cu")
-		(net 3)
-	)
-	(segment
 		(start 170.8403 119.7814)
 		(end 170.9673 119.6036)
@@
 	)
 	(segment
-		(start 163.9061 100.5536)
-		(end 163.2711 101.1886)
-		(width 0.4064)
-		(layer "F.Cu")
-		(net 3)
-	)
-	(segment
 		(start 159.4611 122.6286)
 		(end 159.4611 124.0486)
@@
 		(net 3)
 	)
-	(segment
-		(start 163.9061 100.1786)
-		(end 163.9061 100.5536)
-		(width 0.4064)
-		(layer "F.Cu")
+	(via
+		(at 157.8611 91.0286)
+		(size 0.6)
+		(drill 0.3)
+		(layers "F.Cu" "B.Cu")
+		(free yes)
 		(net 3)
 	)
@@
 	)
 	(via
+		(at 157.8611 83.4086)
+		(size 0.6)
+		(drill 0.3)
+		(layers "F.Cu" "B.Cu")
+		(free yes)
+		(net 3)
+	)
+	(via
 		(at 114.4271 94.8386)
 		(size 0.6)
@@
 	)
 	(segment
-		(start 166.1011 102.4586)
-		(end 168.3511 102.4586)
+		(start 169.6211 98.2036)
+		(end 168.8461 98.2036)
 		(width 0.8128)
 		(layer "F.Cu")
@@
 	)
 	(segment
-		(start 169.6211 99.6646)
-		(end 169.6211 98.6486)
-		(width 0.254)
-		(layer "F.Cu")
-		(net 4)
-	)
-	(segment
-		(start 169.6211 101.1886)
-		(end 169.6211 99.6646)
+		(start 166.4461 100.1786)
+		(end 165.1761 100.1786)
 		(width 0.8128)
 		(layer "F.Cu")
@@
 	)
 	(segment
-		(start 168.3511 102.4586)
-		(end 169.6211 101.1886)
-		(width 0.8128)
-		(layer "F.Cu")
-		(net 4)
-	)
-	(segment
 		(start 119.8371 80.5638)
 		(end 118.4147 79.1414)
@@
 	)
 	(segment
-		(start 141.5795 114.0918)
-		(end 143.2051 114.0918)
-		(width 0.254)
-		(layer "F.Cu")
-		(net 4)
-	)
-	(segment
-		(start 166.4461 100.1786)
-		(end 166.4461 100.5536)
+		(start 169.6211 101.1886)
+		(end 169.6211 98.2036)
 		(width 0.8128)
 		(layer "F.Cu")
@@
 	)
 	(segment
-		(start 126.8731 114.1556)
-		(end 129.4001 114.1556)
-		(width 0.2)
-		(layer "F.Cu")
-		(net 4)
-	)
-	(segment
-		(start 165.9381 101.0616)
-		(end 165.9381 102.0416)
+		(start 169.6211 101.1886)
+		(end 168.6411 102.1686)
 		(width 0.8128)
 		(layer "F.Cu")
@@
 	)
 	(segment
-		(start 124.9171 114.295)
-		(end 124.9361 114.2664)
-		(width 0.254)
-		(layer "F.Cu")
-		(net 4)
-	)
-	(segment
-		(start 165.9381 102.0416)
-		(end 165.8111 102.1686)
+		(start 166.5101 100.2426)
+		(end 166.4461 100.1786)
 		(width 0.8128)
 		(layer "F.Cu")
@@
 	)
 	(segment
-		(start 141.3763 114.295)
-		(end 141.1731 114.0918)
+		(start 141.5795 114.0918)
+		(end 143.2051 114.0918)
 		(width 0.254)
 		(layer "F.Cu")
@@
 	)
 	(segment
-		(start 168.4019 96.8198)
-		(end 168.4019 97.3278)
+		(start 166.5101 102.1686)
+		(end 166.5101 100.2426)
 		(width 0.8128)
 		(layer "F.Cu")
@@
 	)
 	(segment
-		(start 166.4461 100.5536)
-		(end 165.9381 101.0616)
-		(width 0.8128)
+		(start 126.8731 114.1556)
+		(end 129.4001 114.1556)
+		(width 0.2)
 		(layer "F.Cu")
 		(net 4)
 	)
 	(segment
-		(start 169.6211 98.2286)
-		(end 169.6211 99.6646)
-		(width 0.8128)
+		(start 124.9171 114.295)
+		(end 124.9361 114.2664)
+		(width 0.254)
 		(layer "F.Cu")
 		(net 4)
 	)
 	(segment
-		(start 168.4019 97.3278)
-		(end 168.3511 97.3786)
+		(start 168.8461 98.2036)
+		(end 168.0211 97.3786)
 		(width 0.8128)
 		(layer "F.Cu")
@@
 	)
 	(segment
-		(start 166.4461 100.1786)
-		(end 165.1761 100.1786)
-		(width 0.4064)
-		(layer "F.Cu")
-		(net 4)
-	)
-	(segment
-		(start 169.6211 98.6486)
-		(end 169.6211 98.2286)
+		(start 141.3763 114.295)
+		(end 141.1731 114.0918)
 		(width 0.254)
 		(layer "F.Cu")
@@
 	)
 	(segment
-		(start 165.8111 102.1686)
-		(end 166.1011 102.4586)
-		(width 0.8128)
-		(layer "F.Cu")
-		(net 4)
-	)
-	(segment
 		(start 127.0163 114.2664)
 		(end 127.1271 114.1556)
@@
 	)
 	(segment
-		(start 168.3511 97.3786)
-		(end 169.6211 98.6486)
-		(width 0.8128)
-		(layer "F.Cu")
-		(net 4)
-	)
-	(segment
 		(start 140.7667 114.0918)
 		(end 140.7961 114.2664)
@@
 		(net 4)
 	)
+	(segment
+		(start 168.6411 102.1686)
+		(end 166.5101 102.1686)
+		(width 0.8128)
+		(layer "F.Cu")
+		(net 4)
+	)
 	(via
-		(at 168.4019 96.8198)
+		(at 168.0211 97.3786)
 		(size 0.7564)
 		(drill 0.35)
@@
 	)
 	(segment
-		(start 168.4019 96.8198)
-		(end 164.5411 96.8198)
-		(width 0.254)
+		(start 168.0211 97.3786)
+		(end 168.0211 87.2438)
+		(width 0.8128)
 		(layer "B.Cu")
 		(net 4)
@@
 	)
 	(segment
-		(start 164.5411 96.8198)
-		(end 148.2851 113.0758)
+		(start 168.0211 87.2438)
+		(end 168.4019 86.863)
+		(width 0.8128)
+		(layer "B.Cu")
+		(net 4)
+	)
+	(segment
+		(start 148.2851 113.0758)
+		(end 140.5635 113.0758)
 		(width 0.254)
 		(layer "B.Cu")
@@
 	)
 	(segment
-		(start 148.2851 113.0758)
-		(end 140.5635 113.0758)
-		(width 0.254)
-		(layer "B.Cu")
-		(net 4)
-	)
-	(segment
 		(start 163.3219 86.863)
 		(end 155.6003 79.1414)
@@
 	)
 	(segment
-		(start 168.4019 86.863)
-		(end 168.4019 96.8198)
+		(start 174.7011 84.6786)
+		(end 172.5167 86.863)
 		(width 0.8128)
 		(layer "B.Cu")
@@
 	)
 	(segment
-		(start 174.7011 84.6786)
-		(end 172.5167 86.863)
-		(width 0.8128)
+		(start 168.0211 97.3786)
+		(end 163.9823 97.3786)
+		(width 0.254)
+		(layer "B.Cu")
+		(net 4)
+	)
+	(segment
+		(start 163.9823 97.3786)
+		(end 148.2851 113.0758)
+		(width 0.254)
 		(layer "B.Cu")
 		(net 4)
@@
 	)
 	(segment
-		(start 166.4461 94.5786)
-		(end 165.1761 94.5786)
+		(start 167.5211 92.2986)
+		(end 174.5011 99.2786)
 		(width 0.8128)
 		(layer "F.Cu")
@@
 	)
 	(segment
-		(start 161.1511 96.2386)
-		(end 162.2461 96.2386)
+		(start 166.4461 94.5786)
+		(end 165.1761 94.5786)
 		(width 0.8128)
 		(layer "F.Cu")
@@
 	)
 	(segment
-		(start 169.6211 94.3986)
-		(end 174.5011 99.2786)
+		(start 161.1511 96.2386)
+		(end 162.2461 96.2386)
 		(width 0.8128)
 		(layer "F.Cu")
@@
 	)
 	(segment
-		(start 165.8111 92.2986)
-		(end 168.3511 92.2986)
-		(width 0.8128)
-		(layer "F.Cu")
-		(net 7)
-	)
-	(segment
 		(start 163.9061 94.5786)
 		(end 165.1761 94.5786)
@@
 	)
 	(segment
-		(start 168.3511 92.2986)
-		(end 169.6211 93.5686)
-		(width 0.8128)
-		(layer "F.Cu")
-		(net 7)
-	)
-	(segment
 		(start 174.5011 99.2786)
 		(end 178.9887 99.2786)
@@
 	)
 	(segment
-		(start 169.6211 93.5686)
-		(end 169.6211 94.3986)
+		(start 165.8111 92.2986)
+		(end 167.5211 92.2986)
 		(width 0.8128)
 		(layer "F.Cu")

Commit message: replaced 1x01 pinheader's symbol and footprint with kicad library's ones
Parts:
- TP_1V8, TP_3V3, TP_5V0, TP_GLITCH_EN0, TP_GND0, TP_RESET0, TP_TRIGGER2, TP_VTARGET0, X_ANALOG0, X_GLITCH0, X_GLITCH1, X_GLITCH2, X_HPGLITCH2, X_LPGLITCH2, X_TRIGGER0, X_TRIGGER1, X_VCC_EXTERN0: footprint pico-glitcher:1X01 -> Connector_PinHeader_2.54mm:PinHeader_1x01_P2.54mm_Vertical
- turned R2 to -90 degrees
Connections:
- X_VTARGET0 pad 1: unconnected-(X_VTARGET0-Pin_1-Pad1) -> /VTARGET
- X_VTARGET0 pad 2: unconnected-(X_VTARGET0-Pin_2-Pad2) -> /VTARGET
- X_VTARGET0 pad 3: unconnected-(X_VTARGET0-Pin_3-Pad3) -> /VTARGET
Routing:
- net GND: track 71.3 -> 60.4 mm, vias 16 -> 15
- net Net-(X_GLITCH1-Pin_1): track 90.6 -> 87.3 mm

Commit message: replaced 1x02 pinheader's symbol and footprint with kicad library's ones
Parts:
- JMP_VCC_INTERN0: footprint pico-glitcher:1X02 -> Connector_PinHeader_2.54mm:PinHeader_1x02_P2.54mm_Vertical
- moved JMP_VCC_INTERN0 2.55 mm to (174.9, 87.2), turned to 180 degrees
- moved X_VCC_EXTERN0 0.18 mm to (174.9, 79.6)
Connections:
- JMP_VCC_INTERN0 pad 1: VCC -> /JVCC
- JMP_VCC_INTERN0 pad 2: /JVCC -> VCC
Routing:
- net /+1V8: track 39.6 -> 36.6 mm

Commit message: replaced 2x08 pinheader's symbol and footprint with kicad library's ones
Parts:
- X3: footprint pico-glitcher:2X8 -> Connector_PinHeader_2.54mm:PinHeader_2x08_P2.54mm_Vertical
- turned X3 to 0 degrees
