File: schematics/kicad/pico-glitcher.kicad_pcb (KiCad board)
At the start: 2 copper layers, 89.8 x 58.4 mm, 72 parts, among them Q1 IRLML2502, Q2 IRF7807PBF, Q3 TPS 79318, Q4 TPS2041, U1 NH245, U2 NH245, X1 BU-SMA-V, X2 BU-SMA, X3 M08X2

Commit message: replaced power symbols with kicad library's ones
Parts:
- moved R4 2.06 mm to (174.4, 119.7), turned to 180 degrees
- moved R5 0.42 mm to (174.4, 121.8), turned to 180 degrees
- turned R10 to 0 degrees
Connections:
- R4 pad 1: unconnected-(R4-Pad1) -> /HPGLITCH2
Routing:
- net /ANALOG: track 75.6 -> 70.4 mm, vias 2 -> 3
- net +3V3: track 148.7 -> 151.2 mm
- net Net-(Q2-G): track 7.19 -> 5.19 mm
- net /HPGLITCH2: track 102.7 -> 104.1 mm

Commit message: corrected various little things (see details)
 most important thing is that ground plan no longer have themal plane on
 SMD pads. Because some pins are narrowed than the plan minimal width,
 this caused some GND pin to need manual wiring to the ground plan.
Routing:
- net GND: track 60.4 -> 43.5 mm, vias 15 -> 12
- net /LPGLITCH2: track 110.0 -> 108.7 mm
- net /GP7: track 12.4 -> 13.2 mm
- net Net-(U1-B3): track 103.8 -> 103.0 mm
- net /GP6: track 17.1 -> 17.7 mm
- net Net-(X_TRIGGER1-Pin_1): track 77.7 -> 78.1 mm, vias 3 -> 4
- net Net-(X_GLITCH1-Pin_1): vias 3 -> 4

Commit message: replaced SOT-23 symbols with kicad library's ones
Parts:
- Q1: footprint pico-glitcher:SOT23 -> Package_TO_SOT_SMD:SOT-23
- Q3: footprint pico-glitcher:SOT23-5L -> Package_TO_SOT_SMD:SOT-23-5
- moved C2 2.32 mm to (160.4, 84.4), turned to 180 degrees
- turned Q1 to 0 degrees
- turned Q3 to 90 degrees
Routing:
- net /+1V8: track 36.6 -> 37.8 mm

Commit message: replaced 3V3 symbols with kicad library's ones
Parts:
- C1: value 0.01uF -> 10nF
- C2: footprint pico-glitcher:0805 -> Capacitor_SMD:C_0805_2012Metric
Routing:
- net GND: vias 12 -> 10
Changed lines of the file:
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@@
 			)
 		)
-		(property "Value" "0.01uF"
+		(property "Value" "10nF"
 			(at 0 1.43 -90)
 			(layer "F.Fab")
@@
 		)
 	)
-	(footprint "pico-glitcher:0805"
+	(footprint "Capacitor_SMD:C_0805_2012Metric"
 		(layer "F.Cu")
 		(at 160.4011 84.4246 180)
-		(descr "Generic 2012 (0805) package\n\n0.2mm courtyard excess rounded to nearest 0.05mm.")
+		(descr "Capacitor SMD 0805 (2012 Metric), square (rectangular) end terminal, IPC_7351 nominal, (Body size source: IPC-SM-782 page 76, https://www.pcb-3d.com/wordpress/wp-content/uploads/ipc-sm-782a_amendment_1_and_2.pdf, https://docs.google.com/spreadsheets/d/1BsfQQcO9C6DZCsRaXUlFlo91Tg2WpOkGARC1WS5S8t0/edit?usp=sharing), generated with kicad-footprint-generator")
+		(tags "capacitor")
 		(property "Reference" "C2"
-			(at -0.762 -1.016 0)
-			(unlocked yes)
+			(at 0 -1.68 180)
 			(layer "F.SilkS")
 			(effects
 				(font
-					(size 0.773786 0.773786)
-					(thickness 0.039014)
+					(size 1 1)
+					(thickness 0.15)
 				)
-				(justify right top)
 			)
 		)
 		(property "Value" "2.2u"
-			(at -1.016 1.397 0)
-			(unlocked yes)
+			(at 0 1.68 180)
 			(layer "F.Fab")
 			(effects
 				(font
-					(size 0.773786 0.773786)
-					(thickness 0.039014)
+					(size 1 1)
+					(thickness 0.15)
 				)
-				(justify right top)
 			)
 		)
-		(property "Footprint" "pico-glitcher:0805"
-			(at 0 0 360)
+		(property "Footprint" "Capacitor_SMD:C_0805_2012Metric"
+			(at 0 0 180)
+			(unlocked yes)
 			(layer "F.Fab")
 			(hide yes)
@@
 		)
 		(property "Datasheet" ""
-			(at 0 0 360)
+			(at 0 0 180)
+			(unlocked yes)
 			(layer "F.Fab")
 			(hide yes)
@@
 			)
 		)
-		(property "Description" ""
-			(at 0 0 360)
+		(property "Description" "Unpolarized capacitor"
+			(at 0 0 180)
+			(unlocked yes)
 			(layer "F.Fab")
 			(hide yes)
@@
 			)
 		)
+		(property ki_fp_filters "C_*")
 		(sheetname "Root")
 		(sheetfile "pico-glitcher.kicad_sch")
+		(attr smd)
+		(fp_line
+			(start -0.261252 0.735)
+			(end 0.261252 0.735)
+			(stroke
+				(width 0.12)
+				(type solid)
+			)
+			(layer "F.SilkS")
+		)
+		(fp_line
+			(start -0.261252 -0.735)
+			(end 0.261252 -0.735)
+			(stroke
+				(width 0.12)
+				(type solid)
+			)
+			(layer "F.SilkS")
+		)
 		(fp_line
-			(start 1.5 0.8)
-			(end -1.5 0.8)
+			(start 1.7 0.98)
+			(end -1.7 0.98)
 			(stroke
-				(width 0.0508)
+				(width 0.05)
 				(type solid)
 			)
@@
 		)
 		(fp_line
-			(start 1.5 -0.8)
-			(end 1.5 0.8)
+			(start 1.7 -0.98)
+			(end 1.7 0.98)
 			(stroke
-				(width 0.0508)
+				(width 0.05)
 				(type solid)
 			)
@@
 		)
 		(fp_line
-			(start -1.5 0.8)
-			(end -1.5 -0.8)
+			(start -1.7 0.98)
+			(end -1.7 -0.98)
 			(stroke
-				(width 0.0508)
+				(width 0.05)
 				(type solid)
 			)
@@
 		)
 		(fp_line
-			(start -1.5 -0.8)
-			(end 1.5 -0.8)
+			(start -1.7 -0.98)
+			(end 1.7 -0.98)
 			(stroke
-				(width 0.0508)
+				(width 0.05)
 				(type solid)
 			)
 			(layer "F.CrtYd")
 		)
-		(pad "1" smd rect
-			(at -0.9 0 180)
-			(size 0.8 1.2)
+		(fp_line
+			(start 1 0.625)
+			(end -1 0.625)
+			(stroke
+				(width 0.1)
+				(type solid)
+			)
+			(layer "F.Fab")
+		)
+		(fp_line
+			(start 1 -0.625)
+			(end 1 0.625)
+			(stroke
+				(width 0.1)
+				(type solid)
+			)
+			(layer "F.Fab")
+		)
+		(fp_line
+			(start -1 0.625)
+			(end -1 -0.625)
+			(stroke
+				(width 0.1)
+				(type solid)
+			)
+			(layer "F.Fab")
+		)
+		(fp_line
+			(start -1 -0.625)
+			(end 1 -0.625)
+			(stroke
+				(width 0.1)
+				(type solid)
+			)
+			(layer "F.Fab")
+		)
+		(fp_text user "${REFERENCE}"
+			(at 0 0 180)
+			(layer "F.Fab")
+			(effects
+				(font
+					(size 0.5 0.5)
+					(thickness 0.08)
+				)
+			)
+		)
+		(pad "1" smd roundrect
+			(at -0.95 0 180)
+			(size 1 1.45)
 			(layers "F.Cu" "F.Paste" "F.Mask")
+			(roundrect_rratio 0.25)
 			(net 6 "/+1V8")
-			(pinfunction "1")
 			(pintype "passive")
-			(solder_mask_margin 0.1016)
-			(thermal_bridge_angle 0)
 		)
-		(pad "2" smd rect
-			(at 0.9 0 180)
-			(size 0.8 1.2)
+		(pad "2" smd roundrect
+			(at 0.95 0 180)
+			(size 1 1.45)
 			(layers "F.Cu" "F.Paste" "F.Mask")
+			(roundrect_rratio 0.25)
 			(net 3 "GND")
-			(pinfunction "2")
 			(pintype "passive")
-			(solder_mask_margin 0.1016)
-			(thermal_bridge_angle 0)
+		)
+		(model "${KICAD8_3DMODEL_DIR}/Capacitor_SMD.3dshapes/C_0805_2012Metric.wrl"
+			(offset
+				(xyz 0 0 0)
+			)
+			(scale
+				(xyz 1 1 1)
+			)
+			(rotate
+				(xyz 0 0 0)
+			)
 		)
 	)
@@
 	)
 	(via
-		(at 157.8611 91.0286)
+		(at 129.9211 91.0286)
 		(size 0.6)
 		(drill 0.3)
@@
 	)
 	(via
-		(at 130.2511 89.2614)
-		(size 0.6)
-		(drill 0.3)
-		(layers "F.Cu" "B.Cu")
-		(free yes)
-		(net 3)
-	)
-	(via
 		(at 116.2051 101.9506)
 		(size 0.6)
@@
 	)
 	(via
-		(at 130.2511 84.1814)
-		(size 0.6)
-		(drill 0.3)
-		(layers "F.Cu" "B.Cu")
-		(free yes)
-		(net 3)
-	)
-	(via
-		(at 157.8611 83.4086)
+		(at 114.4271 94.8386)
 		(size 0.6)
 		(drill 0.3)
@@
 	)
 	(via
-		(at 114.4271 94.8386)
+		(at 119.2531 100.6806)
 		(size 0.6)
 		(drill 0.3)
@@
 	)
 	(via
-		(at 119.2531 100.6806)
+		(at 148.0311 107.0414)
 		(size 0.6)
 		(drill 0.3)
@@
 	)
 	(via
-		(at 148.0311 107.0414)
+		(at 153.1111 101.9614)
 		(size 0.6)
 		(drill 0.3)
@@
 	)
 	(via
-		(at 153.1111 101.9614)
+		(at 129.9211 85.9486)
 		(size 0.6)
 		(drill 0.3)

Commit message: corrected STO-23(5) footprints and replaced polarized capacitor symbol with kicad library's ones
Parts:
- X1: value BU-SMA-V -> BU-SMA
Changed lines of the file:
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@@
 			)
 		)
-		(property "Description" ""
+		(property "Description" "N-Channel MOSFET IRF9410 and NDS8434 are common, SOIC-8 parts."
 			(at 0 0 90)
 			(layer "F.Fab")
@@
 			)
 		)
-		(property "Description" ""
+		(property "Description" "N-Channel MOSFET - Generic"
 			(at 0 0 0)
 			(unlocked yes)
@@
 			)
 		)
-		(property "Description" ""
+		(property "Description" "RES ARRAY 4 RES 10K OHM 1206   https://www.ctscorp.com/wp-content/uploads/74x.pdf  Manufacturer's datasheet"
 			(at 0 0 180)
 			(layer "F.Fab")
@@
 			)
 		)
-		(property "Description" ""
+		(property "Description" "RES ARRAY 4 RES 10K OHM 1206   https://www.ctscorp.com/wp-content/uploads/74x.pdf  Manufacturer's datasheet"
 			(at 0 0 180)
 			(layer "F.Fab")
@@
 			)
 		)
-		(property "Description" ""
+		(property "Description" "FEMALE SMA CONNECTOR\n\nRadiall\n\ndistributor RS 112-3794"
 			(at 0 0 0)
 			(layer "F.Fab")
@@
 			)
 		)
-		(property "Description" ""
+		(property "Description" "RES ARRAY 4 RES 10K OHM 1206   https://www.ctscorp.com/wp-content/uploads/74x.pdf  Manufacturer's datasheet"
 			(at 0 0 180)
 			(layer "F.Fab")
@@
 			)
 		)
-		(property "Description" ""
+		(property "Description" "RES ARRAY 4 RES 10K OHM 1206   https://www.ctscorp.com/wp-content/uploads/74x.pdf  Manufacturer's datasheet"
 			(at 0 0 180)
 			(layer "F.Fab")
@@
 			)
 		)
-		(property "Value" "BU-SMA-V"
+		(property "Value" "BU-SMA"
 			(at -3.175 5.715 0)
 			(unlocked yes)
@@
 			)
 		)
-		(property "Description" ""
+		(property "Description" "FEMALE SMA CONNECTOR\n\nRadiall\n\ndistributor RS 112-3794"
 			(at 0 0 0)
 			(layer "F.Fab")
@@
 		)
 		(property "Value" "JMP_VCC_INTERN"
-			(at 0 4.87 360)
+			(at 0 4.87 0)
 			(layer "F.Fab")
 			(effects
@@
 		(tags "resistor")
 		(property "Reference" "R10"
-			(at 0 -1.43 360)
+			(at 0 -1.43 0)
 			(layer "F.SilkS")
 			(effects
@@
 		)
 		(property "Value" "150"
-			(at 0 1.43 360)
+			(at 0 1.43 0)
 			(layer "F.Fab")
 			(effects
@@
 		)
 		(fp_text user "${REFERENCE}"
-			(at 0 0 360)
+			(at 0 0 0)
 			(layer "F.Fab")
 			(effects
@@
 			)
 		)
-		(property "Description" ""
+		(property "Description" "RES ARRAY 4 RES 10K OHM 1206   https://www.ctscorp.com/wp-content/uploads/74x.pdf  Manufacturer's datasheet"
 			(at 0 0 180)
 			(layer "F.Fab")
@@
 			)
 		)
-		(property "Description" ""
+		(property "Description" "RES ARRAY 4 RES 10K OHM 1206   https://www.ctscorp.com/wp-content/uploads/74x.pdf  Manufacturer's datasheet"
 			(at 0 0 180)
 			(layer "F.Fab")
@@
 		)
 		(property "Footprint" "pico-glitcher:PANASONIC_C"
-			(at 0 0 -90)
+			(at 0 0 90)
 			(layer "F.Fab")
 			(hide yes)
@@
 		)
 		(property "Datasheet" ""
-			(at 0 0 -90)
+			(at 0 0 90)
 			(layer "F.Fab")
 			(hide yes)
@@
 			)
 		)
-		(property "Description" ""
-			(at 0 0 -90)
+		(property "Description" "Polarized capacitor"
+			(at 0 0 90)
 			(layer "F.Fab")
 			(hide yes)
@@
 			)
 		)
+		(property ki_fp_filters "CP_*")
 		(sheetname "Root")
 		(sheetfile "pico-glitcher.kicad_sch")
@@
 			(layer "F.Fab")
 		)
-		(pad "+" smd rect
-			(at 1.9 0.2 270)
+		(pad "1" smd rect
+			(at -1.8 0.2 270)
 			(size 2.2 0.65)
 			(layers "F.Cu" "F.Paste" "F.Mask")
 			(net 7 "/VTARGET")
-			(pinfunction "+")
 			(pintype "passive")
 			(solder_mask_margin 0.1016)
 			(thermal_bridge_angle 0)
 		)
-		(pad "-" smd rect
-			(at -1.8 0.2 270)
+		(pad "2" smd rect
+			(at 1.9 0.2 270)
 			(size 2.2 0.65)
 			(layers "F.Cu" "F.Paste" "F.Mask")
 			(net 3 "GND")
-			(pinfunction "-")
 			(pintype "passive")
 			(solder_mask_margin 0.1016)
@@
 		(tags "resistor")
 		(property "Reference" "R4"
-			(at 0 1.346 360)
+			(at 0 1.346 0)
 			(layer "F.SilkS")
 			(effects
@@
 		)
 		(property "Value" "1R"
-			(at 0 1.43 360)
+			(at 0 1.43 0)
 			(layer "F.Fab")
 			(effects
@@
 		)
 		(fp_text user "${REFERENCE}"
-			(at 0 0 360)
+			(at 0 0 0)
 			(layer "F.Fab")
 			(effects
@@
 			)
 		)
-		(property "Description" ""
+		(property "Description" "RES ARRAY 4 RES 10K OHM 1206   https://www.ctscorp.com/wp-content/uploads/74x.pdf  Manufacturer's datasheet"
 			(at 0 0 180)
 			(layer "F.Fab")
@@
 		(tags "resistor")
 		(property "Reference" "R5"
-			(at 0 -1.346 360)
+			(at 0 -1.346 0)
 			(layer "F.SilkS")
 			(effects
@@
 		)
 		(property "Value" "10K"
-			(at 0 1.43 360)
+			(at 0 1.43 0)
 			(layer "F.Fab")
 			(effects
@@
 		)
 		(fp_text user "${REFERENCE}"
-			(at 0 0 360)
+			(at 0 0 0)
 			(layer "F.Fab")
 			(effects
@@
 			)
 		)
-		(property "Description" ""
+		(property "Description" "RES ARRAY 4 RES 10K OHM 1206   https://www.ctscorp.com/wp-content/uploads/74x.pdf  Manufacturer's datasheet"
 			(at 0 0 180)
 			(layer "F.Fab")

Commit message: replaced TSSOP-24 footprint with kicad library's ones
Parts:
- U1, U2: footprint pico-glitcher:TSSOP24 -> Package_SO:TSSOP-24_4.4x7.8mm_P0.65mm
- turned U1 to -90 degrees
- turned U2 to -90 degrees
Routing:
- net /GP0: track 19.7 -> 18.2 mm
- net Net-(TP_TRIGGER2-Pin_1): track 92.6 -> 91.6 mm
- net Net-(U1-B3): track 103.0 -> 103.5 mm

Commit message: replaced resistor arrays footprint with kicad library's ones
Parts:
- R12, R13, R14, R15, R16, R17, R18, R19: footprint pico-glitcher:742C083103JP -> Resistor_SMD:R_Array_Concave_4x0603
- turned R12 to -90 degrees
- turned R13 to -90 degrees
- turned R14 to -90 degrees
- turned R15 to -90 degrees
- turned R16 to -90 degrees
- turned R17 to -90 degrees
- turned R18 to -90 degrees
- turned R19 to -90 degrees
Routing:
- net Net-(TP_RESET0-Pin_1): track 121.3 -> 98.9 mm
- net Net-(TP_GLITCH_EN0-Pin_1): track 107.6 -> 101.5 mm
- net Net-(U1-B8): track 44.8 -> 42.0 mm, vias 3 -> 1
- net GND: vias 10 -> 11

Commit message: replaced SOIC-8 footprint with kicad library's one
Parts:
- Q2, Q4: footprint pico-glitcher:SO08 -> Package_SO:SOIC-8_3.9x4.9mm_P1.27mm
- turned Q2 to 180 degrees
- turned Q4 to 90 degrees
Routing:
- net /VTARGET_EN: track 36.4 -> 36.9 mm
