File: schematics/kicad/pico-glitcher.kicad_pcb (KiCad board)
At the start: 2 copper layers, 89.8 x 58.4 mm, 72 parts, among them Q1 IRLML2502, Q2 IRF7807PBF, Q3 TPS 79318, Q4 TPS2041, U1 NH245, U2 NH245, X1 BU-SMA, X2 BU-SMA, X3 M08X2

Commit message: replaced switches' symbol and footprint with kicad library's ones
Parts:
- S1: footprint pico-glitcher:SWITCH-SP3T-SMD -> Button_Switch_SMD:SW_SP3T_PCM13
- S_RST0: value SWITCH-MOMENTARY-2 -> SW_Push_Shielded; footprint pico-glitcher:TACTILE_SWITCH_TALL -> Button_Switch_SMD:SW_Push_1P1T_NO_CK_KSC7xxJ
- moved S_RST0 0.63 mm to (109.3, 125.1), turned to 0 degrees
- moved S1 0.27 mm to (165.8, 78.8), turned to 180 degrees
Connections:
- PICO0 pad RUN: Net-(S_RST0-1) -> Net-(PICO0-PadRUN)
Routing:
- net Net-(S_RST0-1): track 61.1 -> 0.00 mm, vias 4 -> 0
- net Net-(PICO0-PadRUN): track 0.00 -> 54.3 mm, vias 0 -> 4
- net Net-(X3-Pin_1): track 55.6 -> 56.8 mm
- net Net-(U1-B8): track 42.0 -> 42.8 mm
