File: schematics/kicad/pico-glitcher.kicad_sch (KiCad schematic)
At the start: 72 parts, among them Q1 IRLML2502, Q2 IRF7807PBF, Q3 TPS 79318, Q4 TPS2041, U1 NH245, U2 NH245, X1 BU-SMA-V, X2 BU-SMA, X3 M08X2

Commit message: cleaned libraries from unused symbols and footprints
Parts:
- C1, C10, C3, C4, C5, C6, C7, C9: symbol pico-glitcher-eagle-import:0.1UF-0603-25V-10%-X7R-WE -> pico-glitcher:0.1UF-0603-25V-10%-X7R-WE
- C2: symbol pico-glitcher-eagle-import:CAP-0805 -> pico-glitcher:CAP-0805
- C8: symbol pico-glitcher-eagle-import:22UF-POLAR-PANASONIC_C-35V-20% -> pico-glitcher:22UF-POLAR-PANASONIC_C-35V-20%
- D1, D2, D3, D4, D5: symbol pico-glitcher-eagle-import:LED0603 -> pico-glitcher:LED0603
- JMP_VCC_INTERN0: symbol pico-glitcher-eagle-import:CONN_02 -> pico-glitcher:CONN_02
- PICO0: symbol pico-glitcher-eagle-import:RPI_PICO-SMD -> pico-glitcher:RPI_PICO-SMD
- Q1: symbol pico-glitcher-eagle-import:NMOSFETSOT23-GSD -> pico-glitcher:NMOSFETSOT23-GSD
- Q2: symbol pico-glitcher-eagle-import:MOSFET-NCHANNEL-SOIC8 -> pico-glitcher:MOSFET-NCHANNEL-SOIC8
- Q3: symbol pico-glitcher-eagle-import:TPS769XX -> pico-glitcher:TPS769XX
- Q4: symbol pico-glitcher-eagle-import:TPS2041 -> pico-glitcher:TPS2041
- R1, R10, R11, R2, R3, R4, R5, R6, R7, R8, R9: symbol pico-glitcher-eagle-import:10KOHM1/10W1%(0603)0603 -> pico-glitcher:10KOHM1/10W1%(0603)0603
- R12, R13, R14, R15, R16, R17, R18, R19: symbol pico-glitcher-eagle-import:742C083103JP -> pico-glitcher:742C083103JP
- S1: symbol pico-glitcher-eagle-import:SWITCH-SP3T -> pico-glitcher:SWITCH-SP3T
- S_RST0: symbol pico-glitcher-eagle-import:SWITCH-MOMENTARY-2 -> pico-glitcher:SWITCH-MOMENTARY-2
- TP_1V8, TP_3V3, TP_5V0, TP_GLITCH_EN0, TP_GND0, TP_RESET0, TP_TRIGGER2, TP_VTARGET0, X_ANALOG0, X_GLITCH0, X_GLITCH1, X_GLITCH2, X_HPGLITCH2, X_LPGLITCH2, X_TRIGGER0, X_TRIGGER1, X_VCC_EXTERN0: symbol pico-glitcher-eagle-import:M01PTH -> pico-glitcher:M01PTH
- U1, U2: symbol pico-glitcher-eagle-import:NH245-SN74LVC8T245 -> pico-glitcher:NH245-SN74LVC8T245
- X1, X2: symbol pico-glitcher-eagle-import:BU-SMA-V -> pico-glitcher:BU-SMA-V
- X3: symbol pico-glitcher-eagle-import:M08X2 -> pico-glitcher:M08X2
- X_1V8, X_3V3, X_5V0, X_GLITCH_EN0, X_GND0, X_RESET0, X_TRIGGER2, X_VTARGET0: symbol pico-glitcher-eagle-import:M03PTH -> pico-glitcher:M03PTH

Commit message: replaced LEDs symbol and footprint with kicad library's ones
Parts:
- D1, D2, D3, D4, D5: footprint pico-glitcher:LED-0603 -> LED_SMD:LED_0603_1608Metric; symbol pico-glitcher:LED0603 -> Device:LED
Connections:
- net GND: now also D1.1 (K), D2.1 (K), D3.1 (K), D4.1 (K), D5.1 (K); no longer D1.C, D2.C, D3.C, D4.C, D5.C
- net at R7.1: now also D1.2 (A); no longer D1.A
- net at R10.1: now also D5.2 (A); no longer D5.A
- net at R6.1: now also D2.2 (A); no longer D2.A
- net at R8.1: now also D3.2 (A); no longer D3.A
- net at R9.1: now also D4.2 (A); no longer D4.A
Other:
- moved on the sheet: R10, R6, R7, R8, R9

Commit message: replaced 0603 resistor's symbol and footprint with kicad library's ones
Parts:
- R1, R10, R11, R2, R3, R4, R5, R6, R7, R8, R9: footprint pico-glitcher:0603-RES -> Resistor_SMD:R_0603_1608Metric; symbol pico-glitcher:10KOHM1/10W1%(0603)0603 -> Device:R
Connections:
- net GND: now also R2.2; no longer R2.1
- net GP1: now also R6.1; no longer R6.2
- net GP15: now also R8.1; no longer R8.2
- net HPGLITCH2: now also R10.1; no longer R10.2, R4.2
- net LPGLITCH2: now also R7.1; no longer R7.2
- net VTARGET: now also R9.1; no longer R9.2
- net at Q2.4 (G), R5.2: now also R4.2; no longer R4.1
- net at D1.2 (A): now also R7.2; no longer R7.1
- net at D5.2 (A): now also R10.2; no longer R10.1
- net at D2.2 (A): now also R6.2; no longer R6.1
- net at D3.2 (A): now also R8.2; no longer R8.1
- net at D4.2 (A): now also R9.2; no longer R9.1
- net at Q1.1 (G), R3.1: now also R2.1; no longer R2.2

Commit message: replaced 0603 capacitor's symbol and footprint with kicad library's ones
  also: simplified some tracks.
Parts:
- C1, C10, C3, C4, C5, C6, C7, C9: footprint pico-glitcher:0603 -> Capacitor_SMD:C_0603_1608Metric; symbol pico-glitcher:0.1UF-0603-25V-10%-X7R-WE -> Device:C
Changed lines of the file:
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@@
 	)
 	(symbol
-		(lib_id "pico-glitcher:0.1UF-0603-25V-10%-X7R-WE")
-		(at 208.28 71.12 270)
+		(lib_id "Device:C")
+		(at 209.55 71.12 270)
 		(unit 1)
 		(exclude_from_sim no)
@@
 		(dnp no)
 		(property "Reference" "C5"
-			(at 211.201 72.644 0)
+			(at 212.471 72.644 0)
 			(effects
 				(font
@@
 		)
 		(property "Value" "0.1uF"
-			(at 206.121 72.644 0)
+			(at 207.391 72.644 0)
 			(effects
 				(font
@@
 			)
 		)
-		(property "Footprint" "pico-glitcher:0603"
-			(at 208.28 71.12 0)
+		(property "Footprint" "Capacitor_SMD:C_0603_1608Metric"
+			(at 205.74 72.0852 0)
 			(effects
 				(font
@@
 			)
 		)
-		(property "Datasheet" ""
-			(at 208.28 71.12 0)
+		(property "Datasheet" "~"
+			(at 209.55 71.12 0)
 			(effects
 				(font
@@
 			)
 		)
-		(property "Description" ""
-			(at 208.28 71.12 0)
+		(property "Description" "Unpolarized capacitor"
+			(at 209.55 71.12 0)
 			(effects
 				(font
@@
 	)
 	(symbol
-		(lib_id "pico-glitcher:0.1UF-0603-25V-10%-X7R-WE")
-		(at 190.5 71.12 270)
+		(lib_id "Device:C")
+		(at 191.77 71.12 270)
 		(unit 1)
 		(exclude_from_sim no)
@@
 		(dnp no)
 		(property "Reference" "C6"
-			(at 193.421 72.644 0)
+			(at 194.691 72.644 0)
 			(effects
 				(font
@@
 		)
 		(property "Value" "0.1uF"
-			(at 188.341 72.644 0)
+			(at 189.611 72.644 0)
 			(effects
 				(font
@@
 			)
 		)
-		(property "Footprint" "pico-glitcher:0603"
-			(at 190.5 71.12 0)
+		(property "Footprint" "Capacitor_SMD:C_0603_1608Metric"
+			(at 187.96 72.0852 0)
 			(effects
 				(font
@@
 			)
 		)
-		(property "Datasheet" ""
-			(at 190.5 71.12 0)
+		(property "Datasheet" "~"
+			(at 191.77 71.12 0)
 			(effects
 				(font
@@
 			)
 		)
-		(property "Description" ""
-			(at 190.5 71.12 0)
+		(property "Description" "Unpolarized capacitor"
+			(at 191.77 71.12 0)
 			(effects
 				(font
@@
 	)
 	(symbol
-		(lib_id "pico-glitcher:0.1UF-0603-25V-10%-X7R-WE")
-		(at 124.46 220.98 0)
+		(lib_id "Device:C")
+		(at 124.46 219.71 0)
 		(unit 1)
 		(exclude_from_sim no)
@@
 		(dnp no)
 		(property "Reference" "C9"
-			(at 125.984 218.059 0)
+			(at 125.984 216.789 0)
 			(effects
 				(font
@@
 		)
 		(property "Value" "0.1uF"
-			(at 125.984 223.139 0)
+			(at 125.984 221.869 0)
 			(effects
 				(font
@@
 			)
 		)
-		(property "Footprint" "pico-glitcher:0603"
-			(at 124.46 220.98 0)
+		(property "Footprint" "Capacitor_SMD:C_0603_1608Metric"
+			(at 125.4252 223.52 0)
 			(effects
 				(font
@@
 			)
 		)
-		(property "Datasheet" ""
-			(at 124.46 220.98 0)
+		(property "Datasheet" "~"
+			(at 124.46 219.71 0)
 			(effects
 				(font
@@
 			)
 		)
-		(property "Description" ""
-			(at 124.46 220.98 0)
+		(property "Description" "Unpolarized capacitor"
+			(at 124.46 219.71 0)
 			(effects
 				(font
@@
 	)
 	(symbol
-		(lib_id "pico-glitcher:0.1UF-0603-25V-10%-X7R-WE")
-		(at 208.28 144.78 270)
+		(lib_id "Device:C")
+		(at 209.55 144.78 270)
 		(unit 1)
 		(exclude_from_sim no)
@@
 		(dnp no)
 		(property "Reference" "C4"
-			(at 211.201 146.304 0)
+			(at 212.471 146.304 0)
 			(effects
 				(font
@@
 		)
 		(property "Value" "0.1uF"
-			(at 206.121 146.304 0)
+			(at 207.391 146.304 0)
 			(effects
 				(font
@@
 			)
 		)
-		(property "Footprint" "pico-glitcher:0603"
-			(at 208.28 144.78 0)
+		(property "Footprint" "Capacitor_SMD:C_0603_1608Metric"
+			(at 205.74 145.7452 0)
 			(effects
 				(font
@@
 			)
 		)
-		(property "Datasheet" ""
-			(at 208.28 144.78 0)
+		(property "Datasheet" "~"
+			(at 209.55 144.78 0)
 			(effects
 				(font
@@
 			)
 		)
-		(property "Description" ""
-			(at 208.28 144.78 0)
+		(property "Description" "Unpolarized capacitor"
+			(at 209.55 144.78 0)
 			(effects
 				(font
@@
 	)
 	(symbol
-		(lib_id "pico-glitcher:0.1UF-0603-25V-10%-X7R-WE")
-		(at 66.04 45.72 0)
+		(lib_id "Device:C")
+		(at 66.04 44.45 0)
 		(unit 1)
 		(exclude_from_sim no)
@@
 		(dnp no)
 		(property "Reference" "C1"
-			(at 67.564 42.799 0)
+			(at 67.564 41.529 0)
 			(effects
 				(font
@@
 		)
 		(property "Value" "0.01uF"
-			(at 67.564 47.879 0)
+			(at 67.564 46.609 0)
 			(effects
 				(font
@@
 			)
 		)
-		(property "Footprint" "pico-glitcher:0603"
-			(at 66.04 45.72 0)
+		(property "Footprint" "Capacitor_SMD:C_0603_1608Metric"
+			(at 67.0052 48.26 0)
 			(effects
 				(font
@@
 			)
 		)
-		(property "Datasheet" ""
-			(at 66.04 45.72 0)
+		(property "Datasheet" "~"
+			(at 66.04 44.45 0)
 			(effects
 				(font
@@
 			)
 		)
-		(property "Description" ""
-			(at 66.04 45.72 0)
+		(property "Description" "Unpolarized capacitor"
+			(at 66.04 44.45 0)
 			(effects
 				(font
@@
 	)
 	(symbol
-		(lib_id "pico-glitcher:0.1UF-0603-25V-10%-X7R-WE")
-		(at 170.18 236.22 0)
+		(lib_id "Device:C")
+		(at 170.18 234.95 0)
 		(unit 1)
 		(exclude_from_sim no)
@@
 		(dnp no)
 		(property "Reference" "C7"
-			(at 171.704 233.299 0)
+			(at 171.704 232.029 0)
 			(effects
 				(font
@@
 		)
 		(property "Value" "0.1uF"
-			(at 171.704 238.379 0)
+			(at 171.704 237.109 0)
 			(effects
 				(font
@@
 			)
 		)
-		(property "Footprint" "pico-glitcher:0603"
-			(at 170.18 236.22 0)
+		(property "Footprint" "Capacitor_SMD:C_0603_1608Metric"
+			(at 171.1452 238.76 0)
 			(effects
 				(font
@@
 			)
 		)
-		(property "Datasheet" ""
-			(at 170.18 236.22 0)
+		(property "Datasheet" "~"
+			(at 170.18 234.95 0)
 			(effects
 				(font
@@
 			)
 		)
-		(property "Description" ""
-			(at 170.18 236.22 0)
+		(property "Description" "Unpolarized capacitor"
+			(at 170.18 234.95 0)
 			(effects
 				(font
@@
 		)
 		(property "Value" "VCC"
-			(at 203.2 66.04 90)
+			(at 203.2 64.77 90)
 			(effects
 				(font
@@
 	)
 	(symbol
-		(lib_id "pico-glitcher:0.1UF-0603-25V-10%-X7R-WE")
-		(at 25.4 45.72 0)
+		(lib_id "Device:C")
+		(at 25.4 44.45 0)
 		(unit 1)
 		(exclude_from_sim no)
@@
 		(dnp no)
 		(property "Reference" "C10"
-			(at 26.924 42.799 0)
+			(at 26.924 41.529 0)
 			(effects
 				(font
@@
 		)
 		(property "Value" "0.1uF"
-			(at 26.924 47.879 0)
+			(at 26.924 46.609 0)
 			(effects
 				(font
@@
 			)
 		)
-		(property "Footprint" "pico-glitcher:0603"
-			(at 25.4 45.72 0)
+		(property "Footprint" "Capacitor_SMD:C_0603_1608Metric"
+			(at 26.3652 48.26 0)
 			(effects
 				(font
@@
 			)
 		)
-		(property "Datasheet" ""
-			(at 25.4 45.72 0)
+		(property "Datasheet" "~"
+			(at 25.4 44.45 0)
 			(effects
 				(font
@@
 			)
 		)
-		(property "Description" ""
-			(at 25.4 45.72 0)
+		(property "Description" "Unpolarized capacitor"
+			(at 25.4 44.45 0)
 			(effects
 				(font
@@
 		)
 		(property "Value" "+3V3"
-			(at 195.58 71.12 90)
+			(at 198.12 64.77 90)
 			(effects
 				(font
@@
 	)
 	(symbol
-		(lib_id "pico-glitcher:0.1UF-0603-25V-10%-X7R-WE")
-		(at 190.5 144.78 270)
+		(lib_id "Device:C")
+		(at 191.77 144.78 270)
 		(unit 1)
 		(exclude_from_sim no)
@@
 		(dnp no)
 		(property "Reference" "C3"
-			(at 193.421 146.304 0)
+			(at 194.691 146.304 0)
 			(effects
 				(font
@@
 		)
 		(property "Value" "0.1uF"
-			(at 188.341 146.304 0)
+			(at 189.611 146.304 0)
 			(effects
 				(font
@@
 			)
 		)
-		(property "Footprint" "pico-glitcher:0603"
-			(at 190.5 144.78 0)
+		(property "Footprint" "Capacitor_SMD:C_0603_1608Metric"
+			(at 187.96 145.7452 0)
 			(effects
 				(font
@@
 			)
 		)
-		(property "Datasheet" ""
-			(at 190.5 144.78 0)
+		(property "Datasheet" "~"
+			(at 191.77 144.78 0)
 			(effects
 				(font
@@
 			)
 		)
-		(property "Description" ""
-			(at 190.5 144.78 0)
+		(property "Description" "Unpolarized capacitor"
+			(at 191.77 144.78 0)
 			(effects
 				(font

Commit message: replaced 1x03 pinheader's symbol and footprint with kicad library's ones
Parts:
- X_1V8, X_3V3, X_5V0, X_GLITCH_EN0, X_GND0, X_RESET0, X_TRIGGER2, X_VTARGET0: footprint pico-glitcher:1X03 -> Connector_PinHeader_2.54mm:PinHeader_1x03_P2.54mm_Vertical; symbol pico-glitcher:M03PTH -> Connector:Conn_01x03_Pin
Connections:
- net VTARGET: no longer X_VTARGET0.1, X_VTARGET0.2, X_VTARGET0.3

Commit message: replaced 1x01 pinheader's symbol and footprint with kicad library's ones
Parts:
- TP_1V8, TP_3V3, TP_5V0, TP_GLITCH_EN0, TP_GND0, TP_RESET0, TP_TRIGGER2, TP_VTARGET0, X_ANALOG0, X_GLITCH0, X_GLITCH1, X_GLITCH2, X_HPGLITCH2, X_LPGLITCH2, X_TRIGGER0, X_TRIGGER1, X_VCC_EXTERN0: footprint pico-glitcher:1X01 -> Connector_PinHeader_2.54mm:PinHeader_1x01_P2.54mm_Vertical; symbol pico-glitcher:M01PTH -> Connector:Conn_01x01_Pin
Connections:
- net VTARGET: now also X_VTARGET0.1 (Pin_1), X_VTARGET0.2 (Pin_2), X_VTARGET0.3 (Pin_3)

Commit message: replaced 1x02 pinheader's symbol and footprint with kicad library's ones
Parts:
- JMP_VCC_INTERN0: footprint pico-glitcher:1X02 -> Connector_PinHeader_2.54mm:PinHeader_1x02_P2.54mm_Vertical; symbol pico-glitcher:CONN_02 -> Connector:Conn_01x02_Pin
Connections:
- net JVCC: now also JMP_VCC_INTERN0.1 (Pin_1); no longer JMP_VCC_INTERN0.2
- net VCC: now also JMP_VCC_INTERN0.2 (Pin_2); no longer JMP_VCC_INTERN0.1
Other:
- moved on the sheet: JMP_VCC_INTERN0
Changed lines of the file:
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@@
 	)
 	(symbol
-		(lib_id "pico-glitcher:CONN_02")
-		(at 109.22 27.94 180)
+		(lib_id "Connector:Conn_01x02_Pin")
+		(at 106.68 30.48 180)
 		(unit 1)
 		(exclude_from_sim no)
@@
 		(dnp no)
 		(property "Reference" "JMP_VCC_INTERN0"
-			(at 111.76 33.528 0)
+			(at 107.95 30.48 0)
 			(effects
 				(font
 					(size 1.778 1.778)
 				)
-				(justify left bottom)
+				(justify right)
 			)
 		)
 		(property "Value" "JMP_VCC_INTERN"
-			(at 121.92 23.114 0)
+			(at 107.95 27.94 0)
 			(effects
 				(font
 					(size 1.778 1.778)
 				)
-				(justify left bottom)
+				(justify right)
 			)
 		)
-		(property "Footprint" "pico-glitcher:1X02"
-			(at 109.22 27.94 0)
+		(property "Footprint" "Connector_PinHeader_2.54mm:PinHeader_1x02_P2.54mm_Vertical"
+			(at 106.68 30.48 0)
 			(effects
 				(font
@@
 			)
 		)
-		(property "Datasheet" ""
-			(at 109.22 27.94 0)
+		(property "Datasheet" "~"
+			(at 106.68 30.48 0)
 			(effects
 				(font
@@
 			)
 		)
-		(property "Description" ""
-			(at 109.22 27.94 0)
+		(property "Description" "Generic connector, single row, 01x02, script generated"
+			(at 106.68 30.48 0)
 			(effects
 				(font

Commit message: replaced 2x08 pinheader's symbol and footprint with kicad library's ones
Parts:
- X3: footprint pico-glitcher:2X8 -> Connector_PinHeader_2.54mm:PinHeader_2x08_P2.54mm_Vertical; symbol pico-glitcher:M08X2 -> Connector_Generic:Conn_02x08_Odd_Even
Changed lines of the file:
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@@
 	(wire
 		(pts
-			(xy 266.7 175.26) (xy 266.7 144.78)
+			(xy 266.7 175.26) (xy 266.7 142.24)
 		)
 		(stroke
@@
 	(wire
 		(pts
-			(xy 276.86 185.42) (xy 276.86 144.78)
+			(xy 276.86 185.42) (xy 276.86 142.24)
 		)
 		(stroke
@@
 	(wire
 		(pts
-			(xy 264.16 172.72) (xy 264.16 144.78)
+			(xy 264.16 172.72) (xy 264.16 142.24)
 		)
 		(stroke
@@
 	(wire
 		(pts
-			(xy 259.08 144.78) (xy 259.08 149.86)
+			(xy 259.08 142.24) (xy 259.08 149.86)
 		)
 		(stroke
@@
 	(wire
 		(pts
-			(xy 261.62 170.18) (xy 261.62 144.78)
+			(xy 261.62 170.18) (xy 261.62 142.24)
 		)
 		(stroke
@@
 	(wire
 		(pts
-			(xy 271.78 180.34) (xy 271.78 144.78)
+			(xy 271.78 180.34) (xy 271.78 142.24)
 		)
 		(stroke
@@
 	(wire
 		(pts
-			(xy 269.24 177.8) (xy 269.24 144.78)
+			(xy 269.24 177.8) (xy 269.24 142.24)
 		)
 		(stroke
@@
 	(wire
 		(pts
-			(xy 274.32 170.18) (xy 274.32 144.78)
+			(xy 274.32 170.18) (xy 274.32 142.24)
 		)
 		(stroke
@@
 	)
 	(symbol
-		(lib_id "pico-glitcher:M08X2")
-		(at 269.24 137.16 90)
+		(lib_id "Connector_Generic:Conn_02x08_Odd_Even")
+		(at 266.7 137.16 90)
 		(unit 1)
 		(exclude_from_sim no)
@@
 		(dnp no)
 		(property "Reference" "X3"
-			(at 255.27 139.7 0)
+			(at 252.73 139.7 0)
 			(effects
 				(font
@@
 		)
 		(property "Value" "M08X2"
-			(at 281.94 139.7 0)
+			(at 279.4 139.7 0)
 			(effects
 				(font
@@
 			)
 		)
-		(property "Footprint" "pico-glitcher:2X8"
-			(at 269.24 137.16 0)
+		(property "Footprint" "Connector_PinHeader_2.54mm:PinHeader_2x08_P2.54mm_Vertical"
+			(at 266.7 137.16 0)
 			(effects
 				(font
@@
 			)
 		)
-		(property "Datasheet" ""
-			(at 269.24 137.16 0)
+		(property "Datasheet" "~"
+			(at 266.7 137.16 0)
 			(effects
 				(font
@@
 			)
 		)
-		(property "Description" ""
-			(at 269.24 137.16 0)
+		(property "Description" "Generic connector, double row, 02x08, odd/even pin numbering scheme (row 1 odd numbers, row 2 even numbers), script generated (kicad-library-utils/schlib/autogen/connector/)"
+			(at 266.7 137.16 0)
 			(effects
 				(font
