File: schematics/kicad/pico-glitcher.kicad_sch (KiCad schematic)
At the start: 72 parts, among them Q1 IRLML2502, Q2 IRF7807PBF, Q3 TPS 79318, Q4 TPS2041, U1 NH245, U2 NH245, X1 BU-SMA-V, X2 BU-SMA, X3 M08X2

Commit message: replaced power symbols with kicad library's ones
Connections:
- net HPGLITCH2: now also R4.1

Commit message: corrected various little things (see details)
 most important thing is that ground plan no longer have themal plane on
 SMD pads. Because some pins are narrowed than the plan minimal width,
 this caused some GND pin to need manual wiring to the ground plan.
Changed lines of the file:
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@@
 	(paper "User" 325.831 274.218)
 	(junction
+		(at 200.66 119.38)
+		(diameter 0)
+		(color 0 0 0 0)
+	)
+	(junction
 		(at 38.1 165.1)
 		(diameter 0)
@@
 	)
 	(junction
+		(at 200.66 193.04)
+		(diameter 0)
+		(color 0 0 0 0)
+	)
+	(junction
 		(at 217.17 43.18)
 		(diameter 0)
@@
 	(wire
 		(pts
+			(xy 198.12 193.04) (xy 200.66 193.04)
+		)
+		(stroke
+			(width 0)
+			(type default)
+		)
+	)
+	(wire
+		(pts
 			(xy 147.32 243.84) (xy 147.32 241.3)
 		)
@@
 	(wire
 		(pts
+			(xy 200.66 193.04) (xy 203.2 193.04)
+		)
+		(stroke
+			(width 0)
+			(type default)
+		)
+	)
+	(wire
+		(pts
 			(xy 33.02 127) (xy 27.94 127)
 		)
@@
 	(wire
 		(pts
+			(xy 198.12 119.38) (xy 200.66 119.38)
+		)
+		(stroke
+			(width 0)
+			(type default)
+		)
+	)
+	(wire
+		(pts
 			(xy 182.88 111.76) (xy 185.42 111.76)
 		)
@@
 	(wire
 		(pts
+			(xy 200.66 119.38) (xy 203.2 119.38)
+		)
+		(stroke
+			(width 0)
+			(type default)
+		)
+	)
+	(wire
+		(pts
 			(xy 104.14 45.72) (xy 104.14 40.64)
 		)
@@
 		(pin "9"
 		)
+		(pin "13"
+		)
+		(pin "12"
+		)
 		(instances
 			(project ""
@@
 	)
 	(symbol
+		(lib_name "NH245-SN74LVC8T245_1")
 		(lib_id "pico-glitcher:NH245-SN74LVC8T245")
 		(at 200.66 99.06 0)
@@
 		(pin "9"
 		)
+		(pin "12"
+		)
+		(pin "13"
+		)
 		(instances

Commit message: replaced SOT-23 symbols with kicad library's ones
Parts:
- Q1: footprint pico-glitcher:SOT23 -> Package_TO_SOT_SMD:SOT-23
- Q3: footprint pico-glitcher:SOT23-5L -> Package_TO_SOT_SMD:SOT-23-5
Changed lines of the file:
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@@
 			)
 		)
-		(property "Footprint" "pico-glitcher:SOT23-5L"
+		(property "Footprint" "Package_TO_SOT_SMD:SOT-23-5"
 			(at 48.26 40.64 0)
 			(effects
@@
 			)
 		)
-		(property "Footprint" "pico-glitcher:SOT23"
+		(property "Footprint" "Package_TO_SOT_SMD:SOT-23"
 			(at 48.26 162.56 0)
 			(effects

Commit message: replaced 3V3 symbols with kicad library's ones
Parts:
- C1: value 0.01uF -> 10nF
- C2: footprint pico-glitcher:0805 -> Capacitor_SMD:C_0805_2012Metric; symbol pico-glitcher:CAP-0805 -> Device:C
- Q1: footprint Package_TO_SOT_SMD:SOT-23 -> pico-glitcher:SOT23
- Q3: footprint Package_TO_SOT_SMD:SOT-23-5 -> pico-glitcher:SOT23-5L
- X1, X2: footprint pico-glitcher:BU-SMA -> pico-glitcher:BU-SMA-V

Commit message: corrected STO-23(5) footprints and replaced polarized capacitor symbol with kicad library's ones
Parts:
- C8: symbol pico-glitcher:22UF-POLAR-PANASONIC_C-35V-20% -> Device:C_Polarized
- Q1: footprint pico-glitcher:SOT23 -> Package_TO_SOT_SMD:SOT-23
- Q3: footprint pico-glitcher:SOT23-5L -> Package_TO_SOT_SMD:SOT-23-5
- X1: value BU-SMA-V -> BU-SMA; footprint pico-glitcher:BU-SMA-V -> pico-glitcher:BU-SMA
- X2: footprint pico-glitcher:BU-SMA-V -> pico-glitcher:BU-SMA
Connections:
- net GND: now also C8.2; no longer C8.-
- net VTARGET: now also C8.1; no longer C8.+
Changed lines of the file:
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@@
 	)
 	(symbol
-		(lib_id "pico-glitcher:22UF-POLAR-PANASONIC_C-35V-20%")
-		(at 185.42 233.68 0)
+		(lib_id "Device:C_Polarized")
+		(at 185.42 234.95 0)
 		(unit 1)
 		(exclude_from_sim no)
@@
 		(dnp no)
 		(property "Reference" "C8"
-			(at 186.436 233.045 0)
+			(at 186.436 234.315 0)
 			(effects
 				(font
@@
 		)
 		(property "Value" "22uF"
-			(at 186.436 237.871 0)
+			(at 186.436 239.141 0)
 			(effects
 				(font
@@
 		)
 		(property "Footprint" "pico-glitcher:PANASONIC_C"
-			(at 185.42 233.68 0)
+			(at 186.3852 238.76 0)
 			(effects
 				(font
@@
 			)
 		)
-		(property "Datasheet" ""
-			(at 185.42 233.68 0)
+		(property "Datasheet" "~"
+			(at 185.42 234.95 0)
 			(effects
 				(font
@@
 			)
 		)
-		(property "Description" "22µF polarized capacitors\n\nA capacitor is a passive two-terminal electrical component used to store electrical energy temporarily in an electric field."
-			(at 185.42 233.68 0)
+		(property "Description" "Polarized capacitor"
+			(at 185.42 234.95 0)
 			(effects
 				(font
@@
 			)
 		)
-		(pin "+"
+		(pin "2"
 		)
-		(pin "-"
+		(pin "1"
 		)
 		(instances
@@
 			)
 		)
-		(property "Footprint" "pico-glitcher:SOT23-5L"
+		(property "Footprint" "Package_TO_SOT_SMD:SOT-23-5"
 			(at 48.26 40.64 0)
 			(effects
@@
 			)
 		)
-		(property "Value" "BU-SMA-V"
+		(property "Value" "BU-SMA"
 			(at 104.14 160.02 0)
 			(effects
@@
 			)
 		)
-		(property "Footprint" "pico-glitcher:BU-SMA-V"
+		(property "Footprint" "pico-glitcher:BU-SMA"
 			(at 101.6 154.94 0)
 			(effects
@@
 			)
 		)
-		(property "Footprint" "pico-glitcher:SOT23"
+		(property "Footprint" "Package_TO_SOT_SMD:SOT-23"
 			(at 48.26 162.56 0)
 			(effects
@@
 			)
 		)
-		(property "Footprint" "pico-glitcher:BU-SMA-V"
+		(property "Footprint" "pico-glitcher:BU-SMA"
 			(at 127 182.88 0)
 			(effects

Commit message: replaced TSSOP-24 footprint with kicad library's ones
Parts:
- U1, U2: footprint pico-glitcher:TSSOP24 -> Package_SO:TSSOP-24_4.4x7.8mm_P0.65mm
Changed lines of the file:
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@@
 			)
 		)
-		(property "Footprint" "pico-glitcher:TSSOP24"
+		(property "Footprint" "Package_SO:TSSOP-24_4.4x7.8mm_P0.65mm"
 			(at 200.66 172.72 0)
 			(effects
@@
 			)
 		)
-		(property "Footprint" "pico-glitcher:TSSOP24"
+		(property "Footprint" "Package_SO:TSSOP-24_4.4x7.8mm_P0.65mm"
 			(at 200.66 99.06 0)
 			(effects

Commit message: replaced resistor arrays footprint with kicad library's ones
Parts:
- R12, R13, R14, R15, R16, R17, R18, R19: footprint pico-glitcher:742C083103JP -> Resistor_SMD:R_Array_Concave_4x0603
Other:
- moved on the sheet: R12, R13, R14, R15, R16, R17, R18, R19, X_TRIGGER0

Commit message: replaced SOIC-8 footprint with kicad library's one
Parts:
- Q2, Q4: footprint pico-glitcher:SO08 -> Package_SO:SOIC-8_3.9x4.9mm_P1.27mm
Changed lines of the file:
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@@
 			)
 		)
-		(property "Footprint" "pico-glitcher:SO08"
+		(property "Footprint" "Package_SO:SOIC-8_3.9x4.9mm_P1.27mm"
 			(at 58.42 200.66 0)
 			(effects
@@
 			)
 		)
-		(property "Footprint" "pico-glitcher:SO08"
+		(property "Footprint" "Package_SO:SOIC-8_3.9x4.9mm_P1.27mm"
 			(at 147.32 228.6 0)
 			(effects
