File: schematics/kicad/pico-glitcher.kicad_sch (KiCad schematic)
At the start: 72 parts, among them Q1 IRLML2502, Q2 IRF7807PBF, Q3 TPS 79318, Q4 TPS2041, U1 NH245, U2 NH245, X1 BU-SMA, X2 BU-SMA, X3 M08X2

Commit message: replaced switches' symbol and footprint with kicad library's ones
Parts:
- removed S_RST0: SWITCH-MOMENTARY-2, pico-glitcher:TACTILE_SWITCH_TALL, symbol pico-glitcher:SWITCH-MOMENTARY-2
- added S_RST0: SW_Push_Shielded, Button_Switch_SMD:SW_Push_1P1T_NO_CK_KSC7xxJ, symbol Switch:SW_Push
- Q1: footprint Package_TO_SOT_SMD:SOT-23 -> pico-glitcher:SOT23
- Q2, Q4: footprint Package_SO:SOIC-8_3.9x4.9mm_P1.27mm -> pico-glitcher:SO08
- Q3: footprint Package_TO_SOT_SMD:SOT-23-5 -> pico-glitcher:SOT23-5L
- R12, R13, R14, R15, R16, R17, R18, R19: footprint Resistor_SMD:R_Array_Concave_4x0603 -> pico-glitcher:742C083103JP
- S1: footprint pico-glitcher:SWITCH-SP3T-SMD -> Button_Switch_SMD:SW_SP3T_PCM13; symbol pico-glitcher:SWITCH-SP3T -> Switch:SW_SP3T
- U1, U2: footprint Package_SO:TSSOP-24_4.4x7.8mm_P0.65mm -> pico-glitcher:TSSOP24
- X1, X2: footprint pico-glitcher:BU-SMA -> pico-glitcher:BU-SMA-V
Connections:
- net GND: now also S_RST0.2
- net at PICO0.RUN: now also S_RST0.1
Other:
- moved on the sheet: S1
Changed lines of the file:
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@@
 	)
 	(junction
-		(at 88.9 96.52)
-		(diameter 0)
-		(color 0 0 0 0)
-	)
-	(junction
 		(at 219.71 109.22)
 		(diameter 0)
@@
 	(wire
 		(pts
+			(xy 114.3 86.36) (xy 114.3 92.71)
+		)
+		(stroke
+			(width 0)
+			(type default)
+		)
+	)
+	(wire
+		(pts
 			(xy 251.46 111.76) (xy 276.86 111.76)
 		)
@@
 	(wire
 		(pts
-			(xy 88.9 104.14) (xy 88.9 96.52)
-		)
-		(stroke
-			(width 0.1524)
-			(type solid)
-		)
-	)
-	(wire
-		(pts
 			(xy 236.22 132.08) (xy 238.76 132.08)
 		)
@@
 	(wire
 		(pts
+			(xy 113.03 86.36) (xy 114.3 86.36)
+		)
+		(stroke
+			(width 0)
+			(type default)
+		)
+	)
+	(wire
+		(pts
 			(xy 73.66 78.74) (xy 83.82 78.74)
 		)
@@
 	(wire
 		(pts
-			(xy 86.36 104.14) (xy 88.9 104.14)
-		)
-		(stroke
-			(width 0.1524)
-			(type solid)
-		)
-	)
-	(wire
-		(pts
 			(xy 179.07 180.34) (xy 185.42 180.34)
 		)
@@
 	(wire
 		(pts
-			(xy 73.66 104.14) (xy 76.2 104.14)
+			(xy 73.66 104.14) (xy 102.87 104.14)
 		)
 		(stroke
@@
 	(wire
 		(pts
+			(xy 102.87 86.36) (xy 102.87 104.14)
+		)
+		(stroke
+			(width 0.1524)
+			(type solid)
+		)
+	)
+	(wire
+		(pts
 			(xy 43.18 198.12) (xy 43.18 193.04)
 		)
@@
 			)
 		)
-		(property "Footprint" "Package_SO:SOIC-8_3.9x4.9mm_P1.27mm"
+		(property "Footprint" "pico-glitcher:SO08"
 			(at 58.42 200.66 0)
 			(effects
@@
 			)
 		)
-		(property "Footprint" "Package_TO_SOT_SMD:SOT-23-5"
+		(property "Footprint" "pico-glitcher:SOT23-5L"
 			(at 48.26 40.64 0)
 			(effects
@@
 	)
 	(symbol
-		(lib_id "pico-glitcher:SWITCH-SP3T")
+		(lib_id "Switch:SW_SP3T")
 		(at 91.44 30.48 0)
 		(mirror y)
@@
 			)
 		)
-		(property "Footprint" "pico-glitcher:SWITCH-SP3T-SMD"
-			(at 91.44 30.48 0)
+		(property "Footprint" "Button_Switch_SMD:SW_SP3T_PCM13"
+			(at 107.315 26.035 0)
 			(effects
 				(font
@@
 			)
 		)
-		(property "Datasheet" ""
-			(at 91.44 30.48 0)
+		(property "Datasheet" "~"
+			(at 91.44 38.1 0)
 			(effects
 				(font
@@
 			)
 		)
-		(property "Description" ""
+		(property "Description" "Switch, three position, single pole triple throw, 3 position switch, SP3T"
 			(at 91.44 30.48 0)
 			(effects
@@
 			)
 		)
-		(property "Footprint" "Resistor_SMD:R_Array_Concave_4x0603"
+		(property "Footprint" "pico-glitcher:742C083103JP"
 			(at 168.91 113.03 0)
 			(effects
@@
 			)
 		)
-		(property "Footprint" "pico-glitcher:BU-SMA"
+		(property "Footprint" "pico-glitcher:BU-SMA-V"
 			(at 101.6 154.94 0)
 			(effects
@@
 	)
 	(symbol
-		(lib_id "pico-glitcher:SWITCH-MOMENTARY-2")
-		(at 81.28 104.14 0)
-		(unit 1)
-		(exclude_from_sim no)
-		(in_bom yes)
-		(on_board yes)
-		(dnp no)
-		(property "Reference" "S_RST0"
-			(at 78.74 101.6 0)
-			(effects
-				(font
-					(size 1.778 1.5113)
-				)
-				(justify left bottom)
-			)
-		)
-		(property "Value" "SWITCH-MOMENTARY-2"
-			(at 78.74 106.68 0)
-			(effects
-				(font
-					(size 1.778 1.5113)
-				)
-				(justify left bottom)
-			)
-		)
-		(property "Footprint" "pico-glitcher:TACTILE_SWITCH_TALL"
-			(at 81.28 104.14 0)
-			(effects
-				(font
-					(size 1.27 1.27)
-				)
-				(hide yes)
-			)
-		)
-		(property "Datasheet" ""
-			(at 81.28 104.14 0)
-			(effects
-				(font
-					(size 1.27 1.27)
-				)
-				(hide yes)
-			)
-		)
-		(property "Description" ""
-			(at 81.28 104.14 0)
-			(effects
-				(font
-					(size 1.27 1.27)
-				)
-				(hide yes)
-			)
-		)
-		(pin "A2"
-		)
-		(pin "B2"
-		)
-		(instances
-			(project ""
-				(path "/bcbe9e08-2481-468a-b94c-492931ceb6ea"
-					(reference "S_RST0")
-					(unit 1)
-				)
-			)
-		)
-	)
-	(symbol
 		(lib_id "power:GND")
 		(at 38.1 223.52 0)
@@
 			)
 		)
-		(property "Footprint" "Package_SO:SOIC-8_3.9x4.9mm_P1.27mm"
+		(property "Footprint" "pico-glitcher:SO08"
 			(at 147.32 228.6 0)
 			(effects
@@
 			)
 		)
-		(property "Footprint" "Resistor_SMD:R_Array_Concave_4x0603"
+		(property "Footprint" "pico-glitcher:742C083103JP"
 			(at 222.25 121.92 0)
 			(effects
@@
 			)
 		)
-		(property "Footprint" "Resistor_SMD:R_Array_Concave_4x0603"
+		(property "Footprint" "pico-glitcher:742C083103JP"
 			(at 238.76 165.1 0)
 			(effects
@@
 	)
 	(symbol
+		(lib_id "power:GND")
+		(at 114.3 92.71 0)
+		(mirror y)
+		(unit 1)
+		(exclude_from_sim no)
+		(in_bom yes)
+		(on_board yes)
+		(dnp no)
+		(property "Reference" "#GND033"
+			(at 114.3 92.71 0)
+			(effects
+				(font
+					(size 1.27 1.27)
+				)
+				(hide yes)
+			)
+		)
+		(property "Value" "GND"
+			(at 116.84 97.79 0)
+			(effects
+				(font
+					(size 1.778 1.5113)
+				)
+				(justify left bottom)
+			)
+		)
+		(property "Footprint" ""
+			(at 114.3 92.71 0)
+			(effects
+				(font
+					(size 1.27 1.27)
+				)
+				(hide yes)
+			)
+		)
+		(property "Datasheet" ""
+			(at 114.3 92.71 0)
+			(effects
+				(font
+					(size 1.27 1.27)
+				)
+				(hide yes)
+			)
+		)
+		(property "Description" "Power symbol creates a global label with name \"GND\" , ground"
+			(at 114.3 92.71 0)
+			(effects
+				(font
+					(size 1.27 1.27)
+				)
+				(hide yes)
+			)
+		)
+		(pin "1"
+		)
+		(instances
+			(project "pico-glitcher"
+				(path "/bcbe9e08-2481-468a-b94c-492931ceb6ea"
+					(reference "#GND033")
+					(unit 1)
+				)
+			)
+		)
+	)
+	(symbol
 		(lib_id "Device:C")
 		(at 25.4 44.45 0)
@@
 			)
 		)
-		(property "Footprint" "Package_SO:TSSOP-24_4.4x7.8mm_P0.65mm"
+		(property "Footprint" "pico-glitcher:TSSOP24"
 			(at 200.66 172.72 0)
 			(effects
@@
 			)
 		)
-		(property "Footprint" "Resistor_SMD:R_Array_Concave_4x0603"
+		(property "Footprint" "pico-glitcher:742C083103JP"
 			(at 241.3 121.92 0)
 			(effects
@@
 			)
 		)
-		(property "Footprint" "Resistor_SMD:R_Array_Concave_4x0603"
+		(property "Footprint" "pico-glitcher:742C083103JP"
 			(at 162.56 195.58 0)
 			(effects
@@
 	)
 	(symbol
+		(lib_id "Switch:SW_Push")
+		(at 107.95 86.36 0)
+		(unit 1)
+		(exclude_from_sim no)
+		(in_bom yes)
+		(on_board yes)
+		(dnp no)
+		(fields_autoplaced yes)
+		(property "Reference" "S_RST0"
+			(at 107.95 78.74 0)
+			(effects
+				(font
+					(size 1.27 1.27)
+				)
+			)
+		)
+		(property "Value" "SW_Push_Shielded"
+			(at 107.95 81.28 0)
+			(effects
+				(font
+					(size 1.27 1.27)
+				)
+			)
+		)
+		(property "Footprint" "Button_Switch_SMD:SW_Push_1P1T_NO_CK_KSC7xxJ"
+			(at 107.95 81.28 0)
+			(effects
+				(font
+					(size 1.27 1.27)
+				)
+				(hide yes)
+			)
+		)
+		(property "Datasheet" "~"
+			(at 107.95 81.28 0)
+			(effects
+				(font
+					(size 1.27 1.27)
+				)
+				(hide yes)
+			)
+		)
+		(property "Description" "Push button switch, generic, two pins"
+			(at 107.95 86.36 0)
+			(effects
+				(font
+					(size 1.27 1.27)
+				)
+				(hide yes)
+			)
+		)
+		(pin "1"
+		)
+		(pin "2"
+		)
+		(instances
+			(project ""
+				(path "/bcbe9e08-2481-468a-b94c-492931ceb6ea"
+					(reference "S_RST0")
+					(unit 1)
+				)
+			)
+		)
+	)
+	(symbol
 		(lib_id "power:GND")
 		(at 170.18 243.84 0)
@@
 			)
 		)
-		(property "Footprint" "Resistor_SMD:R_Array_Concave_4x0603"
+		(property "Footprint" "pico-glitcher:742C083103JP"
 			(at 168.91 93.98 0)
 			(effects
@@
 			)
 		)
-		(property "Footprint" "Package_TO_SOT_SMD:SOT-23"
+		(property "Footprint" "pico-glitcher:SOT23"
 			(at 48.26 162.56 0)
 			(effects
@@
 			)
 		)
-		(property "Footprint" "Resistor_SMD:R_Array_Concave_4x0603"
+		(property "Footprint" "pico-glitcher:742C083103JP"
 			(at 238.76 180.34 0)
 			(effects
@@
 			)
 		)
-		(property "Footprint" "pico-glitcher:BU-SMA"
+		(property "Footprint" "pico-glitcher:BU-SMA-V"
 			(at 127 182.88 0)
 			(effects
@@
 			)
 		)
-		(property "Footprint" "Package_SO:TSSOP-24_4.4x7.8mm_P0.65mm"
+		(property "Footprint" "pico-glitcher:TSSOP24"
 			(at 200.66 99.06 0)
 			(effects
@@
 			)
 		)
-		(property "Footprint" "Resistor_SMD:R_Array_Concave_4x0603"
+		(property "Footprint" "pico-glitcher:742C083103JP"
 			(at 179.07 195.58 0)
 			(effects
