File: schematics/kicad/pico-glitcher-v2-extension/pico-glitcher-v2.1-extension.kicad_pcb (KiCad board)
At the start: 2 copper layers, 75 x 40 mm, 87 parts, among them J1 Conn_02x10_Odd_Even, J2 Conn_Coaxial, J3 Conn_Coaxial, J4 Conn_01x02_Pin, J5 Conn_01x02_Pin, J6 Conn_01x03_Pin, U1 AD9102BCPZRL7, U2 ADM8829ARTZ-REEL7, U3 ADA4817-1ACP, U4 THS3091DDAR, X1 OB3225125MLDB6SI-00

Commit message: Documentation of pulse-shaping
Other:
- board text added: "Pico Glitcher Pulse Shaping Board v1.0 (c) 2024 Matthias Kesenheimer"
- board text removed: "Pico Glitcher Pulse Shaping Extension v1.0 (c) 2024 Matthias Kesenheimer"

Commit message: correction in documentation
Routing:
- net +5V: track 119.8 -> 120.5 mm
- net GND: vias 31 -> 19
Other:
- board text added: "Pico Glitcher Pulse Shaping Board v1.0 (c) 2025 Matthias Kesenheimer"
- board text removed: "Pico Glitcher Pulse Shaping Board v1.0 (c) 2024 Matthias Kesenheimer"
Changed lines of the file:
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@@
 		)
 	)
-	(gr_text "Pico Glitcher Pulse Shaping Board v1.0\n(c) 2024 Matthias Kesenheimer"
+	(gr_text "Pico Glitcher Pulse Shaping Board v1.0\n(c) 2025 Matthias Kesenheimer"
 		(at 65.25 70.5 0)
 		(layer "F.SilkS")
@@
 	)
 	(via
-		(at 121 85.5)
-		(size 0.6)
-		(drill 0.3)
-		(layers "F.Cu" "B.Cu")
-		(free yes)
-		(net 11)
-	)
-	(via
 		(at 102 88.5)
 		(size 0.6)
@@
 	)
 	(via
-		(at 121 77.5)
-		(size 0.6)
-		(drill 0.3)
-		(layers "F.Cu" "B.Cu")
-		(net 11)
-	)
-	(via
-		(at 120 77.5)
-		(size 0.6)
-		(drill 0.3)
-		(layers "F.Cu" "B.Cu")
-		(net 11)
-	)
-	(via
-		(at 119 76.5)
-		(size 0.6)
-		(drill 0.3)
-		(layers "F.Cu" "B.Cu")
-		(free yes)
-		(net 11)
-	)
-	(via
 		(at 100 78.5)
 		(size 0.6)
@@
 	)
 	(via
-		(at 122 84.5)
-		(size 0.6)
-		(drill 0.3)
-		(layers "F.Cu" "B.Cu")
-		(free yes)
-		(net 11)
-	)
-	(via
 		(at 109.75 71.5)
 		(size 0.6)
@@
 	)
 	(via
-		(at 121 84.5)
-		(size 0.6)
-		(drill 0.3)
-		(layers "F.Cu" "B.Cu")
-		(net 11)
-	)
-	(via
-		(at 122 85.5)
-		(size 0.6)
-		(drill 0.3)
-		(layers "F.Cu" "B.Cu")
-		(free yes)
-		(net 11)
-	)
-	(via
 		(at 110 77)
 		(size 0.6)
@@
 	)
 	(via
-		(at 120 76.5)
-		(size 0.6)
-		(drill 0.3)
-		(layers "F.Cu" "B.Cu")
-		(free yes)
-		(net 11)
-	)
-	(via
 		(at 101 70)
 		(size 0.6)
@@
 	)
 	(via
-		(at 119 77.5)
-		(size 0.6)
-		(drill 0.3)
-		(layers "F.Cu" "B.Cu")
-		(free yes)
-		(net 11)
-	)
-	(via
-		(at 121 76.5)
-		(size 0.6)
-		(drill 0.3)
-		(layers "F.Cu" "B.Cu")
-		(net 11)
-	)
-	(via
 		(at 86.25 92.25)
 		(size 0.6)
@@
 	)
 	(via
-		(at 123 85.5)
-		(size 0.6)
-		(drill 0.3)
-		(layers "F.Cu" "B.Cu")
-		(free yes)
-		(net 11)
-	)
-	(via
 		(at 75.5 104.5)
 		(size 0.6)
@@
 	)
 	(via
-		(at 123 84.5)
-		(size 0.6)
-		(drill 0.3)
-		(layers "F.Cu" "B.Cu")
-		(free yes)
-		(net 11)
-	)
-	(via
 		(at 103.485 77.5)
 		(size 0.6)
@@
 	)
 	(segment
-		(start 124.325 80.215)
-		(end 123.55 80.215)
+		(start 124.1 76.85)
+		(end 125.25 78)
 		(width 0.818)
 		(layer "F.Cu")
@@
 	)
 	(segment
-		(start 123.85 76.85)
-		(end 124.934 77.934)
-		(width 0.818)
-		(layer "F.Cu")
-		(net 12)
-	)
-	(segment
 		(start 79.5 95.5)
 		(end 78.2524 96.7476)
@@
 	)
 	(segment
+		(start 124.785 80.215)
+		(end 123.55 80.215)
+		(width 0.818)
+		(layer "F.Cu")
+		(net 12)
+	)
+	(segment
 		(start 123.85 74.85)
 		(end 123.85 76.85)
@@
 	)
 	(segment
+		(start 123.85 76.85)
+		(end 124.1 76.85)
+		(width 0.818)
+		(layer "F.Cu")
+		(net 12)
+	)
+	(segment
 		(start 105 95.5)
 		(end 115.5 85)
@@
 	)
 	(segment
+		(start 125.25 78)
+		(end 125.25 79.75)
+		(width 0.818)
+		(layer "F.Cu")
+		(net 12)
+	)
+	(segment
 		(start 65.5 100)
 		(end 65.5 103.5)
@@
 	)
 	(segment
+		(start 125.25 79.75)
+		(end 124.785 80.215)
+		(width 0.818)
+		(layer "F.Cu")
+		(net 12)
+	)
+	(segment
 		(start 67.75 99.46)
 		(end 66.04 99.46)
@@
 	)
 	(segment
-		(start 124.934 79.606)
-		(end 124.325 80.215)
-		(width 0.818)
-		(layer "F.Cu")
-		(net 12)
-	)
-	(segment
 		(start 80.450001 101.0616)
 		(end 80.450001 100.189201)
@@
 	)
 	(segment
-		(start 124.934 77.934)
-		(end 124.934 79.606)
-		(width 0.818)
-		(layer "F.Cu")
-		(net 12)
-	)
-	(segment
 		(start 102.7735 74)
 		(end 102.1975 74.576)
@@
 	)
 	(segment
-		(start 116.921 76.579)
-		(end 116.921 79.424682)
+		(start 116.75 76.75)
+		(end 116.75 79.5)
+		(width 0.508)
+		(layer "F.Cu")
+		(net 63)
+	)
+	(segment
+		(start 120.5 73)
+		(end 116.75 76.75)
 		(width 0.508)
 		(layer "F.Cu")
@@
 	)
 	(segment
-		(start 120.5 73)
-		(end 116.921 76.579)
+		(start 117.465 80.215)
+		(end 118.15 80.215)
 		(width 0.508)
 		(layer "F.Cu")
@@
 	)
 	(segment
-		(start 130 74.5)
-		(end 130 76.75)
+		(start 128.5 73)
+		(end 120.5 73)
 		(width 0.508)
 		(layer "F.Cu")
@@
 	)
 	(segment
-		(start 130 78.75)
-		(end 129 77.75)
+		(start 130 74.5)
+		(end 130 76.75)
 		(width 0.508)
 		(layer "F.Cu")
@@
 	)
 	(segment
-		(start 117.711318 80.215)
-		(end 118.15 80.215)
+		(start 130 78.75)
+		(end 129 77.75)
 		(width 0.508)
 		(layer "F.Cu")
@@
 	)
 	(segment
-		(start 128.5 73)
-		(end 120.5 73)
-		(width 0.508)
-		(layer "F.Cu")
-		(net 63)
-	)
-	(segment
-		(start 116.921 79.424682)
-		(end 117.711318 80.215)
+		(start 116.75 79.5)
+		(end 117.465 80.215)
 		(width 0.508)
 		(layer "F.Cu")
@@
 	)
 	(segment
-		(start 127.34 84.5)
+		(start 127.75 84.5)
 		(end 128.75 84.5)
 		(width 0.818)
@@
 	)
 	(segment
-		(start 130 83.25)
-		(end 130 83)
+		(start 128.75 84.5)
+		(end 130 83.25)
 		(width 0.818)
 		(layer "F.Cu")
@@
 	)
 	(segment
-		(start 128.75 84.5)
-		(end 130 83.25)
+		(start 130 83.25)
+		(end 130 83)
 		(width 0.818)
 		(layer "F.Cu")
@@
 	)
 	(segment
-		(start 124.325 81.485)
-		(end 127.34 84.5)
+		(start 123.55 81.485)
+		(end 124.735 81.485)
 		(width 0.818)
 		(layer "F.Cu")
@@
 	)
 	(segment
-		(start 123.55 81.485)
-		(end 124.325 81.485)
+		(start 124.735 81.485)
+		(end 127.75 84.5)
 		(width 0.818)
 		(layer "F.Cu")

Commit message: Bugfixing for Expansion Board schematics
Parts:
- removed C32: 1uF, Capacitor_SMD:C_0805_2012Metric
Connections:
- R18 pad 2: Net-(C32-Pad2) -> /AMPL_VIN+
Routing:
- net /AMPL_VIN+: track 43.3 -> 48.7 mm
- net Net-(C32-Pad2): track 3.52 -> 0.00 mm

Commit message: Solved an issue with Pico Glitcher Pulse Expansion board not storing the calibration
Parts:
- R11: value 200 -> 560
- R12: value 420 -> 120
- R23: value 49.9 -> 1
Connections:
- D3 pad 1: GND -> Net-(D3-K)
- D3 pad 2: Net-(D3-A) -> +3V3
- R10 pad 1: /TRIG -> Net-(D3-K)
- R10 pad 2: Net-(D3-A) -> /TRIG
- R11 pad 2: Net-(JP2-B) -> GND
- R12 pad 1: Net-(JP2-B) -> GND
Routing:
- net Net-(D3-A): track 1.92 -> 0.00 mm
- net (no net): track 0.00 -> 1.92 mm
- net Net-(JP2-B): vias 1 -> 0
- net GND: vias 19 -> 20
Other:
- board text added: "1Ω"
- board text added: "1Ω / 10Ω"
- board text removed: "50Ω"
- board text removed: "50Ω / 10Ω"
Changed lines of the file:
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@@
 	(net 41 "Net-(JP1-B)")
 	(net 42 "Net-(JP1-A)")
-	(net 43 "Net-(D3-A)")
+	(net 43 "Net-(D3-K)")
 	(net 44 "unconnected-(U2-NC-Pad5)")
 	(net 45 "Net-(U2-CAP-)")
@@
 			(layers "F.Cu" "F.Paste" "F.Mask")
 			(roundrect_rratio 0.25)
-			(net 11 "GND")
+			(net 43 "Net-(D3-K)")
 			(pinfunction "K")
 			(pintype "passive")
@@
 			(layers "F.Cu" "F.Paste" "F.Mask")
 			(roundrect_rratio 0.25)
-			(net 43 "Net-(D3-A)")
+			(net 14 "+3V3")
 			(pinfunction "A")
 			(pintype "passive")
@@
 			)
 		)
-		(property "Value" "420"
+		(property "Value" "120"
 			(at 0 1.43 90)
 			(layer "F.Fab")
@@
 			(layers "F.Cu" "F.Paste" "F.Mask")
 			(roundrect_rratio 0.25)
-			(net 51 "Net-(JP2-B)")
+			(net 11 "GND")
 			(pintype "passive")
 		)
@@
 			)
 		)
-		(property "Value" "200"
+		(property "Value" "560"
 			(at 0 1.43 90)
 			(layer "F.Fab")
@@
 			(layers "F.Cu" "F.Paste" "F.Mask")
 			(roundrect_rratio 0.25)
-			(net 51 "Net-(JP2-B)")
+			(net 11 "GND")
 			(pintype "passive")
 		)
@@
 			(layers "F.Cu" "F.Paste" "F.Mask")
 			(roundrect_rratio 0.25)
-			(net 13 "/TRIG")
+			(net 43 "Net-(D3-K)")
 			(pintype "passive")
 		)
@@
 			(layers "F.Cu" "F.Paste" "F.Mask")
 			(roundrect_rratio 0.25)
-			(net 43 "Net-(D3-A)")
+			(net 13 "/TRIG")
 			(pintype "passive")
 		)
@@
 			)
 		)
-		(property "Value" "49.9"
+		(property "Value" "1"
 			(at 0 2.62 90)
 			(layer "F.Fab")
@@
 		(fp_text user "*"
 			(at -1.4732 -2.6518 -90)
+			(unlocked yes)
 			(layer "F.SilkS")
 			(effects
@@
 		(fp_text user "*"
 			(at -1.4732 -2.6518 -90)
-			(unlocked yes)
 			(layer "F.SilkS")
 			(effects
@@
 			)
 		)
-		(fp_text user "*"
-			(at -0.5207 -1.4732 -90)
+		(fp_text user "${REFERENCE}"
+			(at 0 0 -90)
+			(unlocked yes)
 			(layer "F.Fab")
 			(effects
@@
 			)
 		)
-		(fp_text user "${REFERENCE}"
-			(at 0 0 -90)
-			(unlocked yes)
+		(fp_text user "*"
+			(at -0.5207 -1.4732 -90)
 			(layer "F.Fab")
 			(effects
@@
 	)
 	(gr_text "Wup Wup Wup\n(V) (°,,,,°) (V) "
-		(at 137 91.25 0)
+		(at 100.25 103.735 0)
 		(layer "B.SilkS")
 		(effects
 			(font
-				(size 1 1)
-				(thickness 0.15)
+				(size 1.5 1.5)
+				(thickness 0.23)
 			)
 			(justify left bottom mirror)
@@
 		)
 	)
-	(gr_text "50Ω / 10Ω"
+	(gr_text "1Ω / 10Ω"
 		(at 133.5 84.25 90)
 		(layer "F.SilkS")
@@
 		)
 	)
-	(gr_text "50Ω"
-		(at 128.25 95.75 0)
+	(gr_text "1Ω"
+		(at 128.75 95.75 0)
 		(layer "F.SilkS")
 		(effects
@@
 	)
 	(segment
+		(start 96 101)
+		(end 96 102.925)
+		(width 0.254)
+		(layer "F.Cu")
+		(net 0)
+	)
+	(segment
 		(start 102.55 72.05)
 		(end 102.95 72.45)
@@
 	)
 	(via
+		(at 90 74)
+		(size 0.6)
+		(drill 0.3)
+		(layers "F.Cu" "B.Cu")
+		(net 11)
+	)
+	(via
 		(at 114 76.25)
 		(size 0.6)
@@
 	)
 	(segment
-		(start 96 101)
-		(end 96 102.925)
-		(width 0.254)
-		(layer "F.Cu")
-		(net 43)
-	)
-	(segment
 		(start 82.9494 102.1506)
 		(end 79.716601 102.1506)
@@
 		(net 51)
 	)
-	(via
-		(at 90 74)
-		(size 0.6)
-		(drill 0.3)
-		(layers "F.Cu" "B.Cu")
-		(net 51)
-	)
