File: schematics/kicad/pico-glitcher-v2-extension/pico-glitcher-v2.1-extension.kicad_sch (KiCad schematic)
At the start: 87 parts, among them J1 Conn_02x10_Odd_Even, J2 Conn_Coaxial, J3 Conn_Coaxial, J4 Conn_01x02_Pin, J5 Conn_01x02_Pin, J6 Conn_01x03_Pin, U1 AD9102BCPZRL7, U2 ADM8829ARTZ-REEL7, U3 ADA4817-1ACP, U4 THS3091DDAR, X1 OB3225125MLDB6SI-00

Commit message: Bugfixing for Expansion Board schematics
Parts:
- removed C32: 1uF, Capacitor_SMD:C_0805_2012Metric, symbol Device:C
- removed JP2: SolderJumper_2_Bridged, Jumper:SolderJumper-2_P1.3mm_Bridged_Pad1.0x1.5mm, symbol Jumper:SolderJumper_2_Bridged
- R11: value 200 -> 430
- R12: value 420 -> 120
Connections:
- net +3V3: now also D3.2 (A)
- net AMPL_VIN+: now also R18.2
- net GND: now also R11.2, R12.1; no longer D3.1 (K)
- net TRIG: now also R10.2; no longer R10.1
- new net: D3.1 (K), R10.1
Other:
- moved on the sheet: D3, R10

Commit message: Bug fixing and documentation
Parts:
- R11: value 430 -> 560
Other:
- note added: "I = V_INTERM * (1 + (R12 + RV1) / R9) / 50Ω = V_INTERM * [2, 4] / 50Ω"
- note added: "V = +-4mA * (120Ω + 560Ω) + 2.5mA * (560Ω - 120Ω) = -1.6V / + 3.8V"
- note removed: "I = +-2.5V * (1 + (R22 + RV1) / R19) / 50Ω = +-2.5V * [2, 4] / 50Ω = [100mA, 200mA]"
- note removed: "V = +-4mA * (200Ω + 420Ω) = +-2.5V"
Changed lines of the file:
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@@
 		)
 	)
-	(text "I = +-2.5V * (1 + (R22 + RV1) / R19) / 50Ω\n  = +-2.5V * [2, 4] / 50Ω\n  = [100mA, 200mA]"
+	(text "V = +-4mA * (120Ω + 560Ω) + 2.5mA * (560Ω - 120Ω) = -1.6V / + 3.8V"
 		(exclude_from_sim no)
-		(at 252.222 89.662 0)
+		(at 177.292 86.36 0)
 		(effects
 			(font
@@
 		)
 	)
-	(text "V = +-4mA * (200Ω + 420Ω) = +-2.5V"
+	(text "I = V_INTERM * (1 + (R12 + RV1) / R9) / 50Ω\n  = V_INTERM * [2, 4] / 50Ω"
 		(exclude_from_sim no)
-		(at 163.83 93.726 0)
+		(at 253.746 90.424 0)
 		(effects
 			(font
@@
 			)
 		)
-		(property "Value" "430"
+		(property "Value" "560"
 			(at 101.6 105.4099 0)
 			(effects

Commit message: Solved an issue with Pico Glitcher Pulse Expansion board not storing the calibration
Parts:
- R23: value 49.9 -> 1
Changed lines of the file:
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@@
 			)
 		)
-		(property "Value" "49.9"
+		(property "Value" "1"
 			(at 262.89 143.51 90)
 			(effects
