File: schematics/kicad/stm8s-target-v1/stm8s-target-v1.kicad_pcb (KiCad board)
At the start: 2 copper layers, 57 x 25.5 mm, 39 parts, among them J1 ISP_MODE, J10 RESET, J2 VCAP, J3 JMP_3V3, J4 UART, J5 PROGRAM/DEBUG, J6 GPIO, J7 USB_C_Receptacle_USB2.0_16P, J8 Conn_Coaxial, J9 GLITCH_IN, U1 AMS1117-3.3, U2 CH340X, U3 STM8S003F3U

Commit message: refactored findus; renamed scripts (consistent naming scheme); Moved submodules to separate files; fixed an error with arm_multiplexing and the genetic algorithm; added more example scripts; finalized the STM8s target board
Parts:
- removed R11: 100, Resistor_SMD:R_0603_1608Metric
- added D6: D_Small, Diode_SMD:D_SOD-323, F.Cu at (77.3, 83.8)
- added D7: D_Small, Diode_SMD:D_SOD-323, F.Cu at (86.0, 91.2)
- added D8: D_Small, Diode_SMD:D_SOD-323, F.Cu at (86.0, 88.0)
- J3: value JMP_3V3 -> TX/RX
- moved C5 11.3 mm to (96.2, 91.0)
- moved J3 9.46 mm to (92.0, 84.0), turned to 90 degrees
- moved J9 8.75 mm to (100.2, 84.0)
- moved C7 3.48 mm to (94.5, 91.0), turned to 90 degrees
Connections:
- J10 pad 2: /_RESET -> Net-(D8-K)
- J3 pad 1: +3V3 -> /TX
- J3 pad 2: Net-(J3-Pin_2) -> /RX
- J8 pad 1: Net-(J3-Pin_2) -> Net-(J2-Pin_1)
- J9 pad 2: Net-(J3-Pin_2) -> Net-(J2-Pin_1)
- S1 pad 1: /_RESET -> Net-(D6-K)
- S1 pad 4: /_RESET -> Net-(D6-K)
- U3 pad 6: Net-(J3-Pin_2) -> +3V3
Routing:
- net Net-(J3-Pin_2): track 24.6 -> 0.00 mm
- net Net-(J2-Pin_1): track 14.5 -> 33.2 mm
- net Net-(D6-K): track 0.00 -> 11.7 mm
- net /_RESET: track 60.3 -> 49.5 mm
- net +3V3: track 106.6 -> 114.4 mm, vias 1 -> 2
- net Net-(D8-K): track 0.00 -> 4.58 mm
- net /TX: track 67.5 -> 71.9 mm, vias 3 -> 4
- net /RX: track 77.5 -> 80.7 mm, vias 3 -> 4
- net GND: track 199.0 -> 196.9 mm, vias 5 -> 7
- net /_DTR: track 54.1 -> 53.1 mm
Other:
- board text added: "TX RX"
- board text removed: "JMP_3.3V"
