File: schematics/kicad/stm8s-target-v1/stm8s-target-v1.kicad_sch (KiCad schematic)
At the start: 39 parts, among them J1 ISP_MODE, J10 RESET, J2 VCAP, J3 JMP_3V3, J4 UART, J5 PROGRAM/DEBUG, J6 GPIO, J7 USB_C_Receptacle_USB2.0_16P, J8 Conn_Coaxial, J9 GLITCH_IN, U1 AMS1117-3.3, U2 CH340X, U3 STM8S003F3U

Commit message: refactored findus; renamed scripts (consistent naming scheme); Moved submodules to separate files; fixed an error with arm_multiplexing and the genetic algorithm; added more example scripts; finalized the STM8s target board
Parts:
- removed R11: 100, Resistor_SMD:R_0603_1608Metric, symbol Device:R
- added D6, D7, D8: D_Small, Diode_SMD:D_SOD-323, symbol Device:D_Small
- C7: now not fitted
- J3: value JMP_3V3 -> TX/RX
Connections:
- net +3V3: now also U3.6 (VDD); no longer J3.1 (Pin_1)
- net RX: now also J3.2 (Pin_2)
- net TX: now also J3.1 (Pin_1)
- net _DTR: now also D7.1 (K)
- net _RESET: now also D6.2 (A), D8.2 (A); no longer J10.2 (Pin_2), S1.1, S1.4
- net at J2.1 (Pin_1), U3.5 (VCAP): now also J8.1 (In), J9.2 (Pin_2)
- net at JP1.1 (A): now also D7.2 (A)
- new net: D8.1 (K), J10.2 (Pin_2)
- new net: D6.1 (K), S1.1, S1.4
Other:
- moved on the sheet: C5, C6, J10, J2, J8, J9, R8, S1

Commit message: extended STM8Programmer; STM8s glitching is working; fix for issue #18
Parts:
- added R10: 4.7k, Resistor_SMD:R_0603_1608Metric, symbol Device:R
Connections:
- net _CTS: now also R10.1
- net _DTR: now also R10.2
Other:
- note added: "*"
- note added: "* Configure pin 6 as DTR pin"
Changed lines of the file:
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@@
+	)
+	(junction
+		(at 91.44 109.22)
+		(diameter 0)
+		(color 0 0 0 0)
 	)
 	(junction
@@
 	)
 	(junction
+		(at 91.44 99.06)
+		(diameter 0)
+		(color 0 0 0 0)
+	)
+	(junction
 		(at 158.75 110.49)
 		(diameter 0)
@@
 	(wire
 		(pts
+			(xy 91.44 109.22) (xy 97.79 109.22)
+		)
+		(stroke
+			(width 0)
+			(type default)
+		)
+	)
+	(wire
+		(pts
 			(xy 134.62 39.37) (xy 134.62 38.1)
 		)
@@
 	(wire
 		(pts
-			(xy 87.63 109.22) (xy 97.79 109.22)
+			(xy 87.63 109.22) (xy 91.44 109.22)
 		)
 		(stroke
@@
 	(wire
 		(pts
+			(xy 91.44 107.95) (xy 91.44 109.22)
+		)
+		(stroke
+			(width 0)
+			(type default)
+		)
+	)
+	(wire
+		(pts
 			(xy 124.46 110.49) (xy 128.27 110.49)
 		)
@@
 	(wire
 		(pts
+			(xy 91.44 99.06) (xy 91.44 100.33)
+		)
+		(stroke
+			(width 0)
+			(type default)
+		)
+	)
+	(wire
+		(pts
 			(xy 52.07 93.98) (xy 52.07 96.52)
 		)
@@
 	(wire
 		(pts
+			(xy 91.44 99.06) (xy 97.79 99.06)
+		)
+		(stroke
+			(width 0)
+			(type default)
+		)
+	)
+	(wire
+		(pts
 			(xy 120.65 176.53) (xy 118.11 176.53)
 		)
@@
 	(wire
 		(pts
-			(xy 87.63 99.06) (xy 97.79 99.06)
+			(xy 87.63 99.06) (xy 91.44 99.06)
 		)
 		(stroke
@@
 			(width 0.1524)
 			(type solid)
+		)
+	)
+	(text "*"
+		(exclude_from_sim no)
+		(at 88.646 104.394 0)
+		(effects
+			(font
+				(size 1.27 1.27)
+			)
+		)
+	)
+	(text "* Configure pin 6 as DTR pin"
+		(exclude_from_sim no)
+		(at 104.394 85.09 0)
+		(effects
+			(font
+				(size 1.27 1.27)
+			)
 		)
 	)
@@
 					(unit 1)
 				)
+			)
+		)
+	)
+	(symbol
+		(lib_id "Device:R")
+		(at 91.44 104.14 0)
+		(unit 1)
+		(exclude_from_sim no)
+		(in_bom yes)
+		(on_board yes)
+		(dnp no)
+		(property "Reference" "R10"
+			(at 93.726 102.87 0)
+			(effects
+				(font
+					(size 1.27 1.27)
+				)
+				(justify left)
+			)
+		)
+		(property "Value" "4.7k"
+			(at 93.472 105.41 0)
+			(effects
+				(font
+					(size 1.27 1.27)
+				)
+				(justify left)
+			)
+		)
+		(property "Footprint" "Resistor_SMD:R_0603_1608Metric"
+			(at 89.662 104.14 90)
+			(effects
+				(font
+					(size 1.27 1.27)
+				)
+				(hide yes)
+			)
+		)
+		(property "Datasheet" "~"
+			(at 91.44 104.14 0)
+			(effects
+				(font
+					(size 1.27 1.27)
+				)
+				(hide yes)
+			)
+		)
+		(property "Description" "Resistor"
+			(at 91.44 104.14 0)
+			(effects
+				(font
+					(size 1.27 1.27)
+				)
+				(hide yes)
+			)
+		)
+		(pin "1"
+		)
+		(pin "2"
+		)
+		(instances
+			(project "stm8s-target-v1"
+				(path "/688652bf-c811-412a-957f-886210ac2217"
+					(reference "R10")
+					(unit 1)
+				)
