File: schematics/kicad/pulse-shaping-extension-v1/pulse-shaping-extension-v1.kicad_pcb (KiCad board)
At the start: 2 copper layers, 75 x 40 mm, 86 parts, among them J1 Conn_02x10_Odd_Even, J2 Conn_Coaxial, J3 Conn_Coaxial, J4 Conn_01x02_Pin, J5 Conn_01x02_Pin, J6 Conn_01x03_Pin, U1 AD9102BCPZRL7, U2 ADM8829ARTZ-REEL7, U3 ADA4817-1ACP, U4 THS3091DDAR, X1 OB3225125MLDB6SI-00

Commit message: renaming; small changes
Parts:
- removed JP2: SolderJumper_2_Bridged, Jumper:SolderJumper-2_P1.3mm_Bridged_Pad1.0x1.5mm
- added J7: Conn_Coaxial, Connector_Coaxial:SMA_Amphenol_901-144_Vertical, F.Cu at (70.1, 75.0)
- moved TP2 7.27 mm to (75.9, 79.8)
- moved J1 2.21 mm to (67.8, 81.4)
- turned D3 to -90 degrees
- turned R10 to 90 degrees
Routing:
- net Net-(JP2-B): track 5.35 -> 0.00 mm
- net GND: track 528.6 -> 524.1 mm, vias 20 -> 108
- net +3V3: track 150.9 -> 154.2 mm
- net Net-(D3-K): track 0.00 -> 1.92 mm
- net (no net): track 1.92 -> 0.00 mm
- net /SCK: track 23.5 -> 24.7 mm
- net VCC: track 5.52 -> 6.69 mm
- net +5V: track 120.5 -> 119.5 mm
- net /TRIG: track 53.9 -> 54.8 mm
- net /RSTn: track 42.5 -> 43.4 mm
- net /MOSI: track 24.4 -> 25.1 mm
- net /CSn: track 23.6 -> 24.2 mm
Other:
- board text added: "*"
- board text added: "Pico Glitcher Pulse Shaping Board v1.1 (c) 2025 Matthias Kesenheimer"
- board text removed: "Pico Glitcher Pulse Shaping Board v1.0 (c) 2025 Matthias Kesenheimer"
