File: schematics/kicad/pulse-shaping-extension-v1/pulse-shaping-extension-v1.kicad_sch (KiCad schematic)
At the start: 85 parts, among them J1 Conn_02x10_Odd_Even, J2 Conn_Coaxial, J3 Conn_Coaxial, J4 Conn_01x02_Pin, J5 Conn_01x02_Pin, J6 Conn_01x03_Pin, U1 AD9102BCPZRL7, U2 ADM8829ARTZ-REEL7, U3 ADA4817-1ACP, U4 THS3091DDAR, X1 OB3225125MLDB6SI-00

Commit message: renaming; small changes
Parts:
- added J7: Conn_Coaxial, Connector_Coaxial:SMA_Amphenol_901-144_Vertical, symbol Connector:Conn_Coaxial
Connections:
- net GND: now also J7.1 (In), J7.2 (Ext)
Other:
- title: Pico Glitcher v2.1 Pulse Shaping Extension -> Pico Glitcher Pulse Shaping Extension v1.1
Changed lines of the file:
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@@
 	(paper "A4")
 	(title_block
-		(title "Pico Glitcher v2.1 Pulse Shaping Extension")
+		(title "Pico Glitcher Pulse Shaping Extension v1.1")
 		(date "2024-12-27")
 		(rev "v1.0")
@@
 	)
 	(junction
+		(at 227.33 158.75)
+		(diameter 0)
+		(color 0 0 0 0)
+	)
+	(junction
 		(at 124.46 130.81)
 		(diameter 0)
@@
 	(wire
 		(pts
+			(xy 222.25 152.4) (xy 220.98 152.4)
+		)
+		(stroke
+			(width 0)
+			(type default)
+		)
+	)
+	(wire
+		(pts
 			(xy 49.53 160.02) (xy 49.53 161.29)
 		)
@@
 	(wire
 		(pts
+			(xy 227.33 157.48) (xy 227.33 158.75)
+		)
+		(stroke
+			(width 0)
+			(type default)
+		)
+	)
+	(wire
+		(pts
 			(xy 48.26 184.15) (xy 48.26 185.42)
 		)
@@
 	(wire
 		(pts
+			(xy 220.98 158.75) (xy 227.33 158.75)
+		)
+		(stroke
+			(width 0)
+			(type default)
+		)
+	)
+	(wire
+		(pts
 			(xy 52.07 59.69) (xy 72.39 59.69)
 		)
@@
 	(wire
 		(pts
+			(xy 220.98 152.4) (xy 220.98 158.75)
+		)
+		(stroke
+			(width 0)
+			(type default)
+		)
+	)
+	(wire
+		(pts
 			(xy 99.06 99.06) (xy 105.41 99.06)
 		)
@@
 	(wire
 		(pts
+			(xy 227.33 158.75) (xy 227.33 160.02)
+		)
+		(stroke
+			(width 0)
+			(type default)
+		)
+	)
+	(wire
+		(pts
 			(xy 36.83 151.13) (xy 36.83 149.86)
 		)
@@
 	(symbol
 		(lib_id "power:GND")
+		(at 227.33 160.02 0)
+		(unit 1)
+		(exclude_from_sim no)
+		(in_bom yes)
+		(on_board yes)
+		(dnp no)
+		(fields_autoplaced yes)
+		(property "Reference" "#PWR064"
+			(at 227.33 166.37 0)
+			(effects
+				(font
+					(size 1.27 1.27)
+				)
+				(hide yes)
+			)
+		)
+		(property "Value" "GND"
+			(at 227.33 165.1 0)
+			(effects
+				(font
+					(size 1.27 1.27)
+				)
+			)
+		)
+		(property "Footprint" ""
+			(at 227.33 160.02 0)
+			(effects
+				(font
+					(size 1.27 1.27)
+				)
+				(hide yes)
+			)
+		)
+		(property "Datasheet" ""
+			(at 227.33 160.02 0)
+			(effects
+				(font
+					(size 1.27 1.27)
+				)
+				(hide yes)
+			)
+		)
+		(property "Description" "Power symbol creates a global label with name \"GND\" , ground"
+			(at 227.33 160.02 0)
+			(effects
+				(font
+					(size 1.27 1.27)
+				)
+				(hide yes)
+			)
+		)
+		(pin "1"
+		)
+		(instances
+			(project "pico-glitcher-v2.1-extension"
+				(path "/688652bf-c811-412a-957f-886210ac2217"
+					(reference "#PWR064")
+					(unit 1)
+				)
+			)
+		)
+	)
+	(symbol
+		(lib_id "power:GND")
 		(at 135.89 187.96 0)
 		(unit 1)
@@
 					(unit 1)
 				)
+			)
+		)
+	)
+	(symbol
+		(lib_id "Connector:Conn_Coaxial")
+		(at 227.33 152.4 0)
+		(unit 1)
+		(exclude_from_sim no)
+		(in_bom yes)
+		(on_board yes)
+		(dnp no)
+		(property "Reference" "J7"
+			(at 230.124 152.4 0)
+			(effects
+				(font
+					(size 1.27 1.27)
+				)
+				(justify left)
+			)
+		)
+		(property "Value" "Conn_Coaxial"
+			(at 221.488 147.32 0)
+			(effects
+				(font
+					(size 1.27 1.27)
+				)
+				(justify left)
+			)
+		)
+		(property "Footprint" "Connector_Coaxial:SMA_Amphenol_901-144_Vertical"
+			(at 227.33 152.4 0)
+			(effects
+				(font
+					(size 1.27 1.27)
+				)
+				(hide yes)
+			)
+		)
+		(property "Datasheet" "~"
+			(at 227.33 152.4 0)
+			(effects
+				(font
+					(size 1.27 1.27)
+				)
+				(hide yes)
+			)
+		)
+		(property "Description" "coaxial connector (BNC, SMA, SMB, SMC, Cinch/RCA, LEMO, ...)"
+			(at 227.33 152.4 0)
+			(effects
+				(font
+					(size 1.27 1.27)
+				)
+				(hide yes)
+			)
+		)
+		(pin "2"
+		)
+		(pin "1"
+		)
+		(instances
+			(project "pico-glitcher-v2.1-extension"
+				(path "/688652bf-c811-412a-957f-886210ac2217"
+					(reference "J7")
+					(unit 1)
+				)

Commit message: Removed uncessary pull-up resistors for input pins; added pull-up resistors for output pins; removed hardware pull-up resistors for pulse-shaping expansion board; Added new config file for hardware version 2.3 and later; Adopted the documentation; Added new code to support the vtarget switch of hardware version 2.3; Clarified documentation of dead-time
Parts:
- R1, R2, R3: now not fitted
Changed lines of the file:
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@@
 		(in_bom yes)
 		(on_board yes)
-		(dnp no)
+		(dnp yes)
 		(property "Reference" "R1"
 			(at 31.75 26.67 0)
@@
 		(in_bom yes)
 		(on_board yes)
-		(dnp no)
+		(dnp yes)
 		(property "Reference" "R2"
 			(at 26.67 26.67 0)
@@
 		(in_bom yes)
 		(on_board yes)
-		(dnp no)
+		(dnp yes)
 		(fields_autoplaced yes)
 		(property "Reference" "R3"
