File: schematics/kicad/stm8s-target-v1.1/stm8s-target-v1.1.kicad_pcb (KiCad board)
At the start: 2 copper layers, 57 x 25.5 mm, 41 parts, among them J1 ISP_MODE, J10 RESET, J2 VCAP, J3 TX/RX, J4 UART, J5 PROGRAM/DEBUG, J6 GPIO, J7 USB_C_Receptacle_USB2.0_16P, J8 Conn_Coaxial, J9 GLITCH_IN, U1 AMS1117-3.3, U2 CH340X, U3 STM8S003F3U

Commit message: Correction of VTARGET enable; updated schematics
Parts:
- added R10: 4.7k, Resistor_SMD:R_0603_1608Metric, F.Cu at (79.9, 96.3)
Routing:
- net /_CTS: track 50.8 -> 53.2 mm
- net /_DTR: track 53.1 -> 53.9 mm
Other:
- board text added: "Target and UART Board v1.1"
- board text removed: "Target and UART Board v1.0"
