File: schematics/kicad/stm8s-target-v1.1/stm8s-target-v1.1.kicad_sch (KiCad schematic)
At the start: 42 parts, among them J1 ISP_MODE, J10 RESET, J2 VCAP, J3 TX/RX, J4 UART, J5 PROGRAM/DEBUG, J6 GPIO, J7 USB_C_Receptacle_USB2.0_16P, J8 Conn_Coaxial, J9 GLITCH_IN, U1 AMS1117-3.3, U2 CH340X, U3 STM8S003F3U

Commit message: Correction of VTARGET enable; updated schematics
Other:
- title: STM8S Target Board v1 -> STM8S Target Board v1.1
Changed lines of the file:
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@@
 	(paper "A4")
 	(title_block
-		(title "STM8S Target Board v1")
+		(title "STM8S Target Board v1.1")
 		(date "2025-02-21")
-		(rev "v1.0")
+		(rev "v1.1")
 		(company "Faulty Hardware")
 		(comment 1 "Matthias Kesenheimer")
