File: schematics/kicad/pulse-shaping-extension-v1.1/pulse-shaping-extension-v1.1.kicad_pcb (KiCad board)
At the start: 2 copper layers, 75 x 40 mm, 86 parts, among them J1 Conn_02x10_Odd_Even, J2 Conn_Coaxial, J3 Conn_Coaxial, J4 Conn_01x02_Pin, J5 Conn_01x02_Pin, J6 Conn_01x03_Pin, J7 Conn_Coaxial, U1 AD9102BCPZRL7, U2 ADM8829ARTZ-REEL7, U3 ADA4817-1ACP, U4 THS3091DDAR, X1 OB3225125MLDB6SI-00

Commit message: Correction of VTARGET enable; updated schematics
Routing:
- net /AMPL_VIN+: track 48.7 -> 47.7 mm
Other:
- board text removed: "IOUT common ground"

Commit message: Replaced dc-dc converter in pulse shaping expansion board.
Parts:
- removed U2: ADM8829ARTZ-REEL7, footprints:RT_6_ADI
- added U5: ~, Package_TO_SOT_SMD:SOT-363_SC-70-6, F.Cu at (80.4, 102.3)
Routing:
- net Net-(U5-C1-): track 2.81 -> 5.17 mm
- net Net-(U5-C1+): track 5.90 -> 4.04 mm
- net +5V: track 119.5 -> 120.9 mm
Other:
- board text added: "Pico Glitcher Pulse Shaping Board v1.1-r2 (c) 2025 Matthias Kesenheimer"
- board text removed: "Pico Glitcher Pulse Shaping Board v1.1 (c) 2025 Matthias Kesenheimer"
